File: m3_design/assembly_review/battery_entry.kicad_sch (KiCad schematic)
At the start: 20 parts, among them J1 BAT+ / GND / SW / SW, U9 TPS259470LRPWR

Commit message: R2 part-by-part datasheet verification; fix every issue found
All 99 BOM lines / 205 positions checked against manufacturer datasheets
(pinout, land pattern, polarity, part number, 3D orientation); record in
docs/R2_VERIFICATION.md.

Fixes:
- R134/R135: Bourns CRM2512 recommended land (2.45 x 3.7 mm pads, 7.6 mm),
  moved to keep clearance; generic 2512 land had ~45 % of the pad area.
- BOOT0 rerouted out from between the MS5611 pads (TE: do not route
  between pads); 0/45/90 segments instead of 0.1 mm staircases.
- C84 polarity mark on the top side; U12 pin-1 mark.
- AON7524 3D model rotated 180 deg; L1/L2 model height 3.0 mm.
- R84 C705743, R9 C25915, R86 80.6k 0.1% C861568 (80k not orderable);
  every BOM line now has an LCSC code.
- sim_r2: fire with all four servos stalled (FMEA V-15) passes.
- FMEA H-1..H-10 status, redundancy table, firmware requirements,
  README / STATUS / AGENTS updated for R2.

DRC 0 / unconnected 0 / parity 0 / ERC 0, audit OK, actuator contract OK;
diagnostics 173, firmware 112, quality_audit 12 tests pass; sim 135 PASS.

Co-Authored-By: Claude Opus 5.5 (1M context) <noreply@anthropic.com>
Claude-Session: https://claude.ai/code/session_01DdkfTxR7SVyv9xZNmPk9vB
Parts:
- R84: LCSC (none) -> C705743; LCSC Part (none) -> C705743; Manufacturer Yageo -> YAGEO
Changed lines of the file:
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@@
 					(size 1.27 1.27))
 				(justify left)))
-		(property "LCSC" ""
+		(property "LCSC" "C705743"
 			(at 238.76 121.92 0)
 			(hide yes)
@@
 					(reference "R84")
 					(unit 1))))
-		(property "Manufacturer" "Yageo"
+		(property "Manufacturer" "YAGEO"
 			(at 238.76 121.92 0)
 			(hide yes)
@@
 				(font
 					(size 1.27 1.27))))
-		(property "LCSC Part" ""
+		(property "LCSC Part" "C705743"
 			(at 238.76 121.92 0)
 			(hide yes)

Commit message: M3-ASSY-R4: R3 validation fixes, new IMU, fault-tolerant pyro sensing
The board, schematic sheets and footprint library are generated from
R3 (533af8e) by m3_design/r4_build.sh (r4_lib.py, r4_sch.py,
r4_pcb.py). docs/REQUIREMENTS.md states what the board must do;
docs/M3_R4.md records every change, the thirteen evaluation passes
(twelve independent reviews) and the accepted deviations.

- IMU: ST LSM6DSV320X (16 g and 320 g, 4000 dps)
- Pyro: black ARM and orange igniter terminals, eight pyro spacing
  rules in m3.kicad_dru, sense dividers of 2 x 5.1k over 2 x 2k in
  parallel, 4.7k at each ADC pin (R168-R172)
- Pull-pin on a JST PH connector; JLC tooling holes
- Fab: Standard PCBA, 84 BOM lines, 205 placed parts, $80.12 per board
  at five boards (tools/jlc_cost.py); placement rotations verified
- Gate: tools/check.sh DRC 0, unconnected 0, schematic parity 0, ERC 0,
  audit OK; m3_design/check_actuators.py OK

Nothing has been built or measured, and there is no R4 firmware. The
open owner decisions and the bench tests are listed in STATUS.md.

Co-Authored-By: Claude Opus 5.5 <noreply@anthropic.com>
Parts:
- added C87: 2.2uF, rocket:C0603, symbol M3:C
- added C88: 100nF 50V, rocket:C0402, symbol M3:C
- added C89, C95: 22uF 25V X5R 10%, rocket:C_1206_3216Metric, symbol M3:C
- added C96: 10uF 50V X5R 10%, rocket:C_1206_3216Metric, symbol M3:C
- added R165: 470k 1%, rocket:R0402, symbol M3:R
- added R166: 0.33R 1% 2512, rocket:M3_R2512_UR, symbol M3:R
- added R167: 10k 1%, rocket:R_0603_1608Metric, symbol M3:R
- C80: value 1uF 50V X7R 10% -> 10uF 50V X5R 10%; LCSC C1848 -> C13585; LCSC Part C1848 -> C13585; Manufacturer Part CL31B105KBHNNNE -> CL31A106KBHNNNE
- D8: value SMBJ9.0CA -> SMBJ12CA; LCSC C135111 -> C83849; LCSC Part C135111 -> C83849; Manufacturer Diodes Incorporated -> Littelfuse; Manufacturer Part SMBJ9.0CA-13-F -> SMBJ12CA
- R80: value 1M 0.1% -> 470k 1%; LCSC C326730 -> C23178; LCSC Part C326730 -> C23178; Manufacturer Yageo -> UNI-ROYAL(Uniroyal Elec); Manufacturer Part RT0603BRD071ML -> 0603WAF4703T5E
- R81: value 280k 0.1% -> 300k 1%; LCSC C705755 -> C23024; LCSC Part C705755 -> C23024; Manufacturer Yageo -> UNI-ROYAL(Uniroyal Elec); Manufacturer Part RT0603BRD07280KL -> 0603WAF3003T5E
- R83: value 300k 0.1% -> 280k 0.1%; LCSC C705762 -> C705755; LCSC Part C705762 -> C705755; Manufacturer Part RT0603BRD07300KL -> RT0603BRD07280KL
- R89, R92: value 10k 0.1% -> 10k 1%; LCSC C95204 -> C25804; LCSC Part C95204 -> C25804; Manufacturer Yageo -> UNI-ROYAL(Uniroyal Elec); Manufacturer Part RT0603BRD0710KL -> 0603WAF1002T5E
Connections:
- net BAT_ENABLE: now also C87.1, R165.2; no longer J1.4 (SW RETURN)
- net BAT_IN: now also C88.1, C89.1, C95.1, C96.1, R167.1
- net GND: now also C87.2, C88.2, C96.2, R166.2, R167.2
- new net BAT_DAMP: C89.2, C95.2, R166.1
- new net BAT_SW_RETURN: J1.4 (SW RETURN), R165.1
Other:
- note added: "C80 + C96 (2 x 10 uF) at the input; C89 + C95 (2 x 22 uF 25 V X5R) + R166 (0.33 ohm 2512): non-polar RC damper across BAT_IN; R167 (10k) bleeds the input below 2 V within 0.73 s of an unplug (about 1.3 s with the switch closed: wait 2 s). A reverse hot-plug through a 0.1-2 uH, >= 0.03 ohm harness, from <= 2 V left on the input, keeps U9 IN >= -14.6 V and <= 9.2 V/us (TPS25947: -15 V, 10 V/us). No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"
- note added: "C87: EN/UVLO ride-through. (R80+R165)||R81 = 227k charges it (0.4-1.1 s turn-on); R81 alone discharges it (0.66 s), so switch bounce shorter than 0.19/0.33/0.41 s at 6.0/7.4/8.4 V (worst case 0.11/0.21/0.27 s) cannot trip U9 (25-64 us t_D,OFF). UVLO on 4.89-5.05 V, off 4.45-4.61 V."
- note added: "C88: U9 IN bypass at the pin (TI TPS25947 layout guidance); 50 V for the 19.9 V TVS clamp. C80/D8 stay at the terminal."
- note added: "R80 (BAT_IN side) and R165 (EN side) bracket the contact: a chafed SW lead or a battery lead in J1.3/J1.4 puts <= 3.3 V (2S) / 4.9 V (3S) on EN (6.5 V abs max). Power-enable contact, not a main-current break."
- note added: "Reverse battery: R80+R165 (940k) and R82 hold EN/OV injection below 10 uA; C80 and D8 are nonpolar. D8 SMBJ12CA: VBR >= 13.3 V, so a wrong 3S pack (12.6 V) cannot drive it; its 19.9 V clamp is within U9, C80, C88 and Q120 ratings."
- note removed: "R80 precedes the contact and limits wire-fault current. This is a power-enable contact, not a physical main-current break."
- note removed: "Reverse battery: R80/R82 limit EN/OV input injection below10uA; C80 and D8 are nonpolar."
