File: m3_design/assembly_review/battery_entry.kicad_sch (KiCad schematic)
At the start: 28 parts, among them J1 BAT+ / GND / SW / SW, U9 TPS259470LRPWR

Commit message: Validate and harden R5 flight computer CAD
Parts:
- C87: Manufacturer (none) -> Samsung Electro-Mechanics; Manufacturer Part (none) -> CL10A225KO8NNNC
- C88: Manufacturer (none) -> Samsung Electro-Mechanics; Manufacturer Part (none) -> CL05B104KB54PNC
- J1: Manufacturer (none) -> DORABO; Manufacturer Part (none) -> DB128V-5.08-4P-GN-S
- U9: Manufacturer (none) -> Texas Instruments; Manufacturer Part (none) -> TPS259470LRPWR
Changed lines of the file:
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@@
+				(font
+					(size 1.27 1.27))))
+		(property "Manufacturer" "DORABO"
+			(at 71.12 71.12 0)
+			(hide yes)
+			(effects
+				(font
+					(size 1.27 1.27))))
+		(property "Manufacturer Part" "DB128V-5.08-4P-GN-S"
+			(at 71.12 71.12 0)
+			(hide yes)
+			(effects
 				(font
 					(size 1.27 1.27))))
@@
 					(size 1.27 1.27))))
 		(property "LCSC" "C3662793"
+			(at 223.52 76.2 0)
+			(hide yes)
+			(effects
+				(font
+					(size 1.27 1.27))))
+		(property "Manufacturer" "Texas Instruments"
+			(at 223.52 76.2 0)
+			(hide yes)
+			(effects
+				(font
+					(size 1.27 1.27))))
+		(property "Manufacturer Part" "TPS259470LRPWR"
 			(at 223.52 76.2 0)
 			(hide yes)
@@
 					(size 1.27 1.27))
 				(justify left)))
+		(property "Manufacturer" "Samsung Electro-Mechanics"
+			(at 340.36 121.92 0)
+			(hide yes)
+			(effects
+				(font
+					(size 1.27 1.27))
+				(justify left)))
+		(property "Manufacturer Part" "CL10A225KO8NNNC"
+			(at 340.36 121.92 0)
+			(hide yes)
+			(effects
+				(font
+					(size 1.27 1.27))
+				(justify left)))
 		(property "LCSC Part" "C23630"
 			(at 340.36 121.92 0)
@@
 			(at 391.16 121.92 0)
 			(hide yes)
+			(effects
+				(font
+					(size 1.27 1.27))
+				(justify left)))
+		(property "Manufacturer" "Samsung Electro-Mechanics"
+			(at 391.16 121.92 0)
+			(hide yes)
+			(effects
+				(font
+					(size 1.27 1.27))
+				(justify left)))
+		(property "Manufacturer Part" "CL05B104KB54PNC"
+			(at 391.16 121.92 0)
+			(hide yes)

Commit message: Complete R6 flight computer CAD and validated fabrication package
Add protected radio and GPS ports, reset-off port power, compact connectors and single-channel pyro layout. Close independent routing, ground-return and decoupling findings; record zero-error CAD checks and current manufacturing artifacts. Document 100 mm length, IMU stock hold and remaining firmware and hardware qualification.
Parts:
- R165: footprint rocket:R0402 -> rocket:R_0603_1608Metric; LCSC C25790 -> C23178; LCSC Part C25790 -> C23178; Manufacturer Part 0402WGF4703TCE -> 0603WAF4703T5E
- R84: value 1.65k 0.1% -> 750R 0.1%; LCSC C705743 -> C861551; LCSC Part C705743 -> C861551; Manufacturer Part RT0603BRD071K65L -> RT0603BRD07750RL
Changed lines of the file:
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@@
 		(title "07 | Battery input, contact and protection")
 		(date "2026-09-07")
-		(rev "M3-ASSY-R4")
+		(rev "M3-ASSY-R6")
 		(company "Single-board M3 candidate; full system incomplete"))
 	(text "07 | Battery input, contact and protection"
@@
 					(size 1.27 1.27))
 				(justify left)))
-		(property "Value" "1.65k 0.1%"
+		(property "Value" "750R 0.1%"
 			(at 241.29999999999998 123.19000000000001 0)
 			(effects
@@
 					(size 1.27 1.27))
 				(justify left)))
-		(property "LCSC" "C705743"
+		(property "LCSC" "C861551"
 			(at 238.76 121.92 0)
 			(hide yes)
@@
 				(font
 					(size 1.27 1.27))))
-		(property "Manufacturer Part" "RT0603BRD071K65L"
+		(property "Manufacturer Part" "RT0603BRD07750RL"
 			(at 238.76 121.92 0)
 			(hide yes)
@@
 				(font
 					(size 1.27 1.27))))
-		(property "LCSC Part" "C705743"
+		(property "LCSC Part" "C861551"
 			(at 238.76 121.92 0)
 			(hide yes)
@@
 					(size 1.27 1.27))
 				(justify left)))
-		(property "Footprint" "rocket:R0402"
+		(property "Footprint" "rocket:R_0603_1608Metric"
 			(at 370.84 121.92 0)
 			(hide yes)
@@
 					(size 1.27 1.27))
 				(justify left)))
-		(property "LCSC" "C25790"
+		(property "LCSC" "C23178"
 			(at 370.84 121.92 0)
 			(hide yes)
@@
 					(size 1.27 1.27))
 				(justify left)))
-		(property "LCSC Part" "C25790"
+		(property "LCSC Part" "C23178"
 			(at 370.84 121.92 0)
 			(hide yes)
@@
 					(size 1.27 1.27))
 				(justify left)))
-		(property "Manufacturer Part" "0402WGF4703TCE"
+		(property "Manufacturer Part" "0603WAF4703T5E"
 			(at 370.84 121.92 0)
 			(hide yes)
