File: m3_design/assembly_review/camera_uart.kicad_sch (KiCad schematic)
At the start: 12 parts, among them U12 TXU0202DCUR, U13 TPS70933DBVR

Commit message: M3-ASSY-R2: merge servos, dual fused pyro, arming, pull-pin and buzzer
Adds every remaining hardware function to the single M3 board (46 x 238 mm,
203 positions / 178 fitted parts, 14 sheets):

- Actuator power switch: back-to-back AON6403 from the battery input, gated
  by the U9 logic path so the one external switch still controls everything.
- Single-deploy dual pyro (owner ruling 2026-09-25): two AON7524 channels on
  two independently fused buses (FMEA H-5), separate 4-pos ARM and igniter
  terminals, per-bus arm sense, continuity, cold pull-up (H-1), gate networks
  per MARGIN_PRESCRIPTION P0-1/P0-2, PE3/PE6 sentinels (LED_RED -> PE8).
- Four servos (1 k series, pull-downs, SRV05-4), clamped pull-pin (PC14),
  MLT-8530 buzzer (PA5; pad mapping from the maker spec).
- Backup altimeter fully isolated by ruling: no interface on the board.
- New AON7524 footprint from AOS PO-00047 rev I; U12 LCSC code added.
- tools/export_fab.py (Gerber/drill zip, JLC BOM + CPL); m3_design/
  check_actuators.py (arming break / gate-network contract from PCB nets).

CAD checks only: tools/check.sh DRC 0 / unconnected 0 / parity 0 / ERC 0,
audit OK. No bench, simulation or flight evidence; no R2 firmware yet.

Co-Authored-By: Claude Opus 5.5 <noreply@anthropic.com>
Parts:
- U12: LCSC (none) -> C5186957; LCSC Part (none) -> C5186957
Changed lines of the file:
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@@
 				(font
 					(size 1.27 1.27))))
-		(property "LCSC" ""
+		(property "LCSC" "C5186957"
 			(at 259.08 78.74 0)
 			(hide yes)
@@
 				(font
 					(size 1.27 1.27))))
-		(property "LCSC Part" ""
+		(property "LCSC Part" "C5186957"
 			(at 259.08 78.74 0)
 			(hide yes)

Commit message: M3-ASSY-R3: 1k 1% resistors to JLC Basic, regenerate fab package, cost gate
R74/R77/R100/R101/R103: C22548 (Yageo RC0603FR-071KL) -> C21190 (UNI-ROYAL
0603WAF1001T5E), same 1k 1% 100 ppm 0.1 W 75 V 0603 land. The 100 nF C1591 ->
C14663 swap was not made: C128/C140 sit on the pyro outputs and no DC-bias data
exists for the replacement, so the line stays extended either way.
jlc_orient: C21190 via a same-footprint donor (EasyEDA API returned 403).
export_fab: 75 lines, 180 placed, no missing LCSC, no unverified rotation.
jlc_stock --boards 5: short only U4 ICM-45686 (JLC stock 0, protected).
jlc_cost: parts $54.94/board at 5 boards, 48 unique extended codes (gate counts
codes, not rows). check.sh all zero.

Co-Authored-By: Claude Opus 5.5 <noreply@anthropic.com>
Parts:
- R100, R101, R103: LCSC C22548 -> C21190; LCSC Part C22548 -> C21190; Manufacturer Yageo -> UNI-ROYAL(Uniroyal Elec); Manufacturer Part RC0603FR-071KL -> 0603WAF1001T5E
Changed lines of the file:
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@@
 					(size 1.27 1.27))
 				(justify left)))
-		(property "LCSC" "C22548"
+		(property "LCSC" "C21190"
 			(at 91.44 193.04 0)
 			(hide yes)
@@
 					(reference "R100")
 					(unit 1))))
-		(property "Manufacturer" "Yageo"
+		(property "Manufacturer" "UNI-ROYAL(Uniroyal Elec)"
 			(at 91.44 193.04 0)
 			(hide yes)
@@
 				(font
 					(size 1.27 1.27))))
-		(property "Manufacturer Part" "RC0603FR-071KL"
+		(property "Manufacturer Part" "0603WAF1001T5E"
 			(at 91.44 193.04 0)
 			(hide yes)
@@
 				(font
 					(size 1.27 1.27))))
-		(property "LCSC Part" "C22548"
+		(property "LCSC Part" "C21190"
 			(at 91.44 193.04 0)
 			(hide yes)
@@
 					(size 1.27 1.27))
 				(justify left)))
-		(property "LCSC" "C22548"
+		(property "LCSC" "C21190"
 			(at 172.72 193.04 0)
 			(hide yes)
@@
 					(reference "R101")
 					(unit 1))))
-		(property "Manufacturer" "Yageo"
-			(at 172.72 193.04 0)
-			(hide yes)
-			(effects
-				(font
-					(size 1.27 1.27))))
-		(property "Manufacturer Part" "RC0603FR-071KL"
-			(at 172.72 193.04 0)
-			(hide yes)
-			(effects
-				(font
-					(size 1.27 1.27))))
-		(property "LCSC Part" "C22548"
+		(property "Manufacturer" "UNI-ROYAL(Uniroyal Elec)"
+			(at 172.72 193.04 0)
+			(hide yes)
+			(effects
+				(font
+					(size 1.27 1.27))))
+		(property "Manufacturer Part" "0603WAF1001T5E"
+			(at 172.72 193.04 0)
+			(hide yes)
+			(effects
+				(font
+					(size 1.27 1.27))))
+		(property "LCSC Part" "C21190"
 			(at 172.72 193.04 0)
 			(hide yes)
@@
 					(size 1.27 1.27))
 				(justify left)))
-		(property "LCSC" "C22548"
+		(property "LCSC" "C21190"
 			(at 147.32 137.16 0)
 			(hide yes)
@@
 					(reference "R103")
 					(unit 1))))
-		(property "Manufacturer" "Yageo"
-			(at 147.32 137.16 0)
-			(hide yes)
-			(effects
-				(font
-					(size 1.27 1.27))))
-		(property "Manufacturer Part" "RC0603FR-071KL"
-			(at 147.32 137.16 0)
-			(hide yes)
-			(effects
-				(font
-					(size 1.27 1.27))))
-		(property "LCSC Part" "C22548"
-			(at 147.32 137.16 0)
-			(hide yes)
+		(property "Manufacturer" "UNI-ROYAL(Uniroyal Elec)"
+			(at 147.32 137.16 0)
+			(hide yes)
+			(effects
+				(font
+					(size 1.27 1.27))))
+		(property "Manufacturer Part" "0603WAF1001T5E"
+			(at 147.32 137.16 0)
+			(hide yes)
+			(effects
+				(font
+					(size 1.27 1.27))))
+		(property "LCSC Part" "C21190"
+			(at 147.32 137.16 0)
+			(hide yes)

Commit message: M3-ASSY-R4: R3 validation fixes, new IMU, fault-tolerant pyro sensing
The board, schematic sheets and footprint library are generated from
R3 (533af8e) by m3_design/r4_build.sh (r4_lib.py, r4_sch.py,
r4_pcb.py). docs/REQUIREMENTS.md states what the board must do;
docs/M3_R4.md records every change, the thirteen evaluation passes
(twelve independent reviews) and the accepted deviations.

- IMU: ST LSM6DSV320X (16 g and 320 g, 4000 dps)
- Pyro: black ARM and orange igniter terminals, eight pyro spacing
  rules in m3.kicad_dru, sense dividers of 2 x 5.1k over 2 x 2k in
  parallel, 4.7k at each ADC pin (R168-R172)
- Pull-pin on a JST PH connector; JLC tooling holes
- Fab: Standard PCBA, 84 BOM lines, 205 placed parts, $80.12 per board
  at five boards (tools/jlc_cost.py); placement rotations verified
- Gate: tools/check.sh DRC 0, unconnected 0, schematic parity 0, ERC 0,
  audit OK; m3_design/check_actuators.py OK

Nothing has been built or measured, and there is no R4 firmware. The
open owner decisions and the bench tests are listed in STATUS.md.

Co-Authored-By: Claude Opus 5.5 <noreply@anthropic.com>
Parts:
- C90, C93: LCSC C1591 -> C14663; LCSC Part C1591 -> C14663; Manufacturer Samsung Electro-Mechanics -> YAGEO; Manufacturer Part CL10B104KB8NNNC -> CC0603KRX7R9BB104
- R102: value 10k 0.1% -> 10k 1%; LCSC C95204 -> C25804; LCSC Part C95204 -> C25804; Manufacturer Yageo -> UNI-ROYAL(Uniroyal Elec); Manufacturer Part RT0603BRD0710KL -> 0603WAF1002T5E
Changed lines of the file:
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@@
 		(title "09 | Camera UART, separate supply domains")
 		(date "2026-09-07")
-		(rev "M3-ASSY-R3")
+		(rev "M3-ASSY-R4")
 		(company "Single-board M3 candidate; full system incomplete"))
 	(text "09 | Camera UART, separate supply domains"
@@
 					(size 1.27 1.27))
 				(justify left)))
-		(property "Value" "10k 0.1%"
+		(property "Value" "10k 1%"
 			(at 332.74 138.42999999999998 0)
 			(effects
@@
 					(size 1.27 1.27))
 				(justify left)))
-		(property "LCSC" "C95204"
+		(property "LCSC" "C25804"
 			(at 330.2 137.16 0)
 			(hide yes)
@@
 					(reference "R102")
 					(unit 1))))
-		(property "Manufacturer" "Yageo"
+		(property "Manufacturer" "UNI-ROYAL(Uniroyal Elec)"
 			(at 330.2 137.16 0)
 			(hide yes)
@@
 				(font
 					(size 1.27 1.27))))
-		(property "Manufacturer Part" "RT0603BRD0710KL"
+		(property "Manufacturer Part" "0603WAF1002T5E"
 			(at 330.2 137.16 0)
 			(hide yes)
@@
 				(font
 					(size 1.27 1.27))))
-		(property "LCSC Part" "C95204"
+		(property "LCSC Part" "C25804"
 			(at 330.2 137.16 0)
 			(hide yes)
@@
 					(size 1.27 1.27))
 				(justify left)))
-		(property "LCSC" "C1591"
+		(property "LCSC" "C14663"
 			(at 213.36 137.16 0)
 			(hide yes)
@@
 					(reference "C90")
 					(unit 1))))
-		(property "Manufacturer" "Samsung Electro-Mechanics"
+		(property "Manufacturer" "YAGEO"
 			(at 213.36 137.16 0)
 			(hide yes)
@@
 				(font
 					(size 1.27 1.27))))
-		(property "Manufacturer Part" "CL10B104KB8NNNC"
+		(property "Manufacturer Part" "CC0603KRX7R9BB104"
 			(at 213.36 137.16 0)
 			(hide yes)
@@
 				(font
 					(size 1.27 1.27))))
-		(property "LCSC Part" "C1591"
+		(property "LCSC Part" "C14663"
 			(at 213.36 137.16 0)
 			(hide yes)
@@
 					(size 1.27 1.27))
 				(justify left)))
-		(property "LCSC" "C1591"
+		(property "LCSC" "C14663"
 			(at 269.24 137.16 0)
 			(hide yes)
@@
 					(reference "C93")
 					(unit 1))))
-		(property "Manufacturer" "Samsung Electro-Mechanics"
+		(property "Manufacturer" "YAGEO"
 			(at 269.24 137.16 0)
 			(hide yes)
@@
 				(font
 					(size 1.27 1.27))))
-		(property "Manufacturer Part" "CL10B104KB8NNNC"
+		(property "Manufacturer Part" "CC0603KRX7R9BB104"
 			(at 269.24 137.16 0)
 			(hide yes)
@@
 				(font
 					(size 1.27 1.27))))
-		(property "LCSC Part" "C1591"
+		(property "LCSC Part" "C14663"
 			(at 269.24 137.16 0)
 			(hide yes)
