File: m3_design/assembly_review/camera_uart.kicad_sch (KiCad schematic)
At the start: 12 parts, among them U12 TXU0202DCUR, U13 TPS70933DBVR

Commit message: Validate and harden R5 flight computer CAD
Parts:
- added C100: 100nF, rocket:C0402, symbol M3:C
Connections:
- net 3V3: now also C100.1
- net GND: now also C100.2
Changed lines of the file:
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@@
 	(title_block
 		(title "09 | Camera UART, separate supply domains")
-		(date "2026-09-07")
-		(rev "M3-ASSY-R4")
+		(date "2026-10-12")
+		(rev "M3-ASSY-R5")
 		(company "Single-board M3 candidate; full system incomplete"))
 	(text "09 | Camera UART, separate supply domains"
@@
 	(sheet_instances
 		(path "/"
-			(page "9"))))
+			(page "9")))
+	(symbol
+		(lib_id "M3:C")
+		(at 81.2800 165.1000 0)
+		(unit 1)
+		(in_bom yes)
+		(on_board yes)
+		(dnp no)
+		(property "Reference" "C100"
+			(at 83.8200 163.8300 0)
+			(effects
+				(font
+					(size 1.27 1.27))
+				(justify left)))
+		(property "Value" "100nF"
+			(at 83.8200 166.3700 0)
+			(effects
+				(font
+					(size 1.27 1.27))
+				(justify left)))
+		(property "Footprint" "rocket:C0402"
+			(at 81.2800 165.1000 0)
+			(hide yes)
+			(effects
+				(font
+					(size 1.27 1.27))
+				(justify left)))
+		(property "Datasheet" ""
+			(at 81.2800 165.1000 0)
+			(hide yes)
+			(effects
+				(font
+					(size 1.27 1.27))
+				(justify left)))
+		(property "LCSC" "C1525"
+			(at 81.2800 165.1000 0)
+			(hide yes)
+			(effects
+				(font
+					(size 1.27 1.27))
+				(justify left)))
+		(property "Manufacturer" "Samsung Electro-Mechanics"
+			(at 81.2800 165.1000 0)
+			(hide yes)
+			(effects
+				(font
+					(size 1.27 1.27))
+				(justify left)))
+		(property "Manufacturer Part" "CL05B104KO5NNNC"
+			(at 81.2800 165.1000 0)
+			(hide yes)
+			(effects
+				(font
+					(size 1.27 1.27))
+				(justify left)))
+		(instances
+			(project "m3"
+				(path "/6007a7db-6a58-5660-8beb-956dea045ff8/3918f78b-b8e6-50fb-8165-8fdc93a836ab"
+					(reference "C100")
+					(unit 1)))))
+	(wire (pts (xy 81.28 161.2900) (xy 73.6600 161.2900)) (stroke (width 0) (type default)))
+	(global_label "3V3" (shape passive) (at 73.6600 161.2900 0) (effects (font (size 1.05 1.05)) (justify right)))
+	(wire (pts (xy 81.28 168.9100) (xy 73.6600 168.9100)) (stroke (width 0) (type default)))
+	(global_label "GND" (shape passive) (at 73.6600 168.9100 0) (effects (font (size 1.05 1.05)) (justify right)))
+)

Commit message: Complete R6 flight computer CAD and validated fabrication package
Add protected radio and GPS ports, reset-off port power, compact connectors and single-channel pyro layout. Close independent routing, ground-return and decoupling findings; record zero-error CAD checks and current manufacturing artifacts. Document 100 mm length, IMU stock hold and remaining firmware and hardware qualification.
Parts:
- C100: value 100nF -> 100nF 50V X7R 10%; LCSC C1525 -> C307331; LCSC Part (none) -> C307331; Manufacturer Part CL05B104KO5NNNC -> CL05B104KB54PNC
Changed lines of the file:
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@@
 		(title "09 | Camera UART, separate supply domains")
 		(date "2026-10-12")
-		(rev "M3-ASSY-R5")
+		(rev "M3-ASSY-R6")
 		(company "Single-board M3 candidate; full system incomplete"))
 	(text "09 | Camera UART, separate supply domains"
@@
 					(size 1.27 1.27))
 				(justify left)))
-		(property "Value" "100nF"
+		(property "Value" "100nF 50V X7R 10%"
 			(at 83.8200 166.3700 0)
 			(effects
@@
 					(size 1.27 1.27))
 				(justify left)))
-		(property "LCSC" "C1525"
+		(property "LCSC" "C307331"
 			(at 81.2800 165.1000 0)
 			(hide yes)
@@
 					(size 1.27 1.27))
 				(justify left)))
-		(property "Manufacturer Part" "CL05B104KO5NNNC"
+		(property "Manufacturer Part" "CL05B104KB54PNC"
 			(at 81.2800 165.1000 0)
 			(hide yes)
@@
 				(path "/6007a7db-6a58-5660-8beb-956dea045ff8/3918f78b-b8e6-50fb-8165-8fdc93a836ab"
 					(reference "C100")
-					(unit 1)))))
+					(unit 1))))		(property "LCSC Part" "C307331"
+			(at 0 0 0)
+			(hide yes)
+			(effects
+				(font
+					(size 1.27 1.27))
+				(justify left)))
+)
 	(wire (pts (xy 81.28 161.2900) (xy 73.6600 161.2900)) (stroke (width 0) (type default)))
 	(global_label "3V3" (shape passive) (at 73.6600 161.2900 0) (effects (font (size 1.05 1.05)) (justify right)))
