File: m3_design/assembly_review/logic_power_path.kicad_sch (KiCad schematic)
At the start: 16 parts, among them U10 TPS2553DBVR, U11 TPS2121RUXR

Commit message: R2 part-by-part datasheet verification; fix every issue found
All 99 BOM lines / 205 positions checked against manufacturer datasheets
(pinout, land pattern, polarity, part number, 3D orientation); record in
docs/R2_VERIFICATION.md.

Fixes:
- R134/R135: Bourns CRM2512 recommended land (2.45 x 3.7 mm pads, 7.6 mm),
  moved to keep clearance; generic 2512 land had ~45 % of the pad area.
- BOOT0 rerouted out from between the MS5611 pads (TE: do not route
  between pads); 0/45/90 segments instead of 0.1 mm staircases.
- C84 polarity mark on the top side; U12 pin-1 mark.
- AON7524 3D model rotated 180 deg; L1/L2 model height 3.0 mm.
- R84 C705743, R9 C25915, R86 80.6k 0.1% C861568 (80k not orderable);
  every BOM line now has an LCSC code.
- sim_r2: fire with all four servos stalled (FMEA V-15) passes.
- FMEA H-1..H-10 status, redundancy table, firmware requirements,
  README / STATUS / AGENTS updated for R2.

DRC 0 / unconnected 0 / parity 0 / ERC 0, audit OK, actuator contract OK;
diagnostics 173, firmware 112, quality_audit 12 tests pass; sim 135 PASS.

Co-Authored-By: Claude Opus 5.5 (1M context) <noreply@anthropic.com>
Claude-Session: https://claude.ai/code/session_01DdkfTxR7SVyv9xZNmPk9vB
Parts:
- R86: value 80k 0.1% -> 80.6k 0.1%; LCSC (none) -> C861568; LCSC Part (none) -> C861568; Manufacturer Vishay Dale Thin Film -> YAGEO; Manufacturer Part PTN0603Y8002BST1 -> RT0603BRD0780K6L
Changed lines of the file:
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@@
 					(size 1.27 1.27))
 				(justify left)))
-		(property "Value" "80k 0.1%"
+		(property "Value" "80.6k 0.1%"
 			(at 261.62 128.27 0)
 			(effects
@@
 					(size 1.27 1.27))
 				(justify left)))
-		(property "LCSC" ""
+		(property "LCSC" "C861568"
 			(at 259.08 127 0)
 			(hide yes)
@@
 					(reference "R86")
 					(unit 1))))
-		(property "Manufacturer" "Vishay Dale Thin Film"
+		(property "Manufacturer" "YAGEO"
 			(at 259.08 127 0)
 			(hide yes)
@@
 				(font
 					(size 1.27 1.27))))
-		(property "Manufacturer Part" "PTN0603Y8002BST1"
+		(property "Manufacturer Part" "RT0603BRD0780K6L"
 			(at 259.08 127 0)
 			(hide yes)
@@
 				(font
 					(size 1.27 1.27))))
-		(property "LCSC Part" ""
+		(property "LCSC Part" "C861568"
 			(at 259.08 127 0)
 			(hide yes)

Commit message: Make R2 orderable: stocked drop-ins, JLC placement corrections, ordering guide
- Stock (JLC assembly API): U8 AP63200 -> AP63300WU-7 (same TSOT26 pinout,
  VFB, fsw), L3 -> SRP5030T-6R8M (same body/land, AP63300 Table 1), C77
  100p -> 47p (Table 1), C84 25SVPF330M -> 35SVPK330M (same OS-CON F12).
  Every BOM line now has JLC stock for 5 boards except U6 SAM-M10Q
  (consign / Global Sourcing; DigiKey has stock).
- tools/jlc_orient.py matches each footprint pad-by-pad to the LCSC/EasyEDA
  footprint of its LCSC code; export_fab.py applies the rotation/offset.
  Without it U7, U8, U10, U11, U12, U13, D121 and LED2 would be rotated.
- tools/jlc_stock.py: repeatable stock check; fab/stock_check.json.
- JLC_Assembly field: U6 consign note, J2/J123 hand-cut from one 1x40 strip.
- docs/ORDERING.md: PCB options, PCBA, preview checklist, off-board parts.

DRC 0 / unconnected 0 / parity 0 / ERC 0, audit OK; contract OK;
tests 173/112/12 pass; sim 135 PASS.

Co-Authored-By: Claude Opus 5.5 (1M context) <noreply@anthropic.com>
Claude-Session: https://claude.ai/code/session_01DdkfTxR7SVyv9xZNmPk9vB
Parts:
- C84: value 330uF 25V -> 330uF 35V; LCSC C178367 -> C178373; LCSC Part (none) -> C178373; Manufacturer (none) -> Panasonic; Manufacturer Part (none) -> 35SVPK330M
Changed lines of the file:
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@@
 				(font
 					(size 1.27 1.27))))
-		(property "Value" "330uF 25V"
+		(property "Value" "330uF 35V"
 			(at 360.68 119.38 0)
 			(effects
@@
 				(font
 					(size 1.27 1.27))))
-		(property "LCSC" "C178367"
+		(property "LCSC" "C178373"
 			(at 360.68 127 0)
 			(hide yes)
+			(effects
+				(font
+					(size 1.27 1.27))))
+		(property "LCSC Part" "C178373"
+			(at 360.68 127 0)
+			(hide yes)
+			(effects
+				(font
+					(size 1.27 1.27))))
+		(property "Manufacturer" "Panasonic"
+			(at 360.68 127 0)
+			(hide yes)
+			(effects
+				(font
+					(size 1.27 1.27))))
+		(property "Manufacturer Part" "35SVPK330M"
+			(at 360.68 127 0)
+			(hide yes)

Commit message: M3-ASSY-R4: R3 validation fixes, new IMU, fault-tolerant pyro sensing
The board, schematic sheets and footprint library are generated from
R3 (533af8e) by m3_design/r4_build.sh (r4_lib.py, r4_sch.py,
r4_pcb.py). docs/REQUIREMENTS.md states what the board must do;
docs/M3_R4.md records every change, the thirteen evaluation passes
(twelve independent reviews) and the accepted deviations.

- IMU: ST LSM6DSV320X (16 g and 320 g, 4000 dps)
- Pyro: black ARM and orange igniter terminals, eight pyro spacing
  rules in m3.kicad_dru, sense dividers of 2 x 5.1k over 2 x 2k in
  parallel, 4.7k at each ADC pin (R168-R172)
- Pull-pin on a JST PH connector; JLC tooling holes
- Fab: Standard PCBA, 84 BOM lines, 205 placed parts, $80.12 per board
  at five boards (tools/jlc_cost.py); placement rotations verified
- Gate: tools/check.sh DRC 0, unconnected 0, schematic parity 0, ERC 0,
  audit OK; m3_design/check_actuators.py OK

Nothing has been built or measured, and there is no R4 firmware. The
open owner decisions and the bench tests are listed in STATUS.md.

Co-Authored-By: Claude Opus 5.5 <noreply@anthropic.com>
Parts:
- C83: LCSC C1591 -> C14663; LCSC Part C1591 -> C14663; Manufacturer Samsung Electro-Mechanics -> YAGEO; Manufacturer Part CL10B104KB8NNNC -> CC0603KRX7R9BB104
- R87: value 44.2k 0.1% -> 47k 1%; LCSC C861410 -> C25819; LCSC Part C861410 -> C25819; Manufacturer Yageo -> UNI-ROYAL(Uniroyal Elec); Manufacturer Part RT0603BRD0744K2L -> 0603WAF4702T5E
- R88, R90, R91: value 10k 0.1% -> 10k 1%; LCSC C95204 -> C25804; LCSC Part C95204 -> C25804; Manufacturer Yageo -> UNI-ROYAL(Uniroyal Elec); Manufacturer Part RT0603BRD0710KL -> 0603WAF1002T5E
Changed lines of the file:
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@@
 		(title "08 | USB limit, source mux and hold-up")
 		(date "2026-09-07")
-		(rev "M3-ASSY-R3")
+		(rev "M3-ASSY-R4")
 		(company "Single-board M3 candidate; full system incomplete"))
 	(text "08 | USB limit, source mux and hold-up"
@@
 					(size 1.27 1.27))
 				(justify left)))
-		(property "LCSC" "C1591"
+		(property "LCSC" "C14663"
 			(at 43.18 127 0)
 			(hide yes)
@@
 					(reference "C83")
 					(unit 1))))
-		(property "Manufacturer" "Samsung Electro-Mechanics"
+		(property "Manufacturer" "YAGEO"
 			(at 43.18 127 0)
 			(hide yes)
@@
 				(font
 					(size 1.27 1.27))))
-		(property "Manufacturer Part" "CL10B104KB8NNNC"
+		(property "Manufacturer Part" "CC0603KRX7R9BB104"
 			(at 43.18 127 0)
 			(hide yes)
@@
 				(font
 					(size 1.27 1.27))))
-		(property "LCSC Part" "C1591"
+		(property "LCSC Part" "C14663"
 			(at 43.18 127 0)
 			(hide yes)
@@
 					(size 1.27 1.27))
 				(justify left)))
-		(property "Value" "44.2k 0.1%"
+		(property "Value" "47k 1%"
 			(at 210.82 181.60999999999999 0)
 			(effects
@@
 					(size 1.27 1.27))
 				(justify left)))
-		(property "LCSC" "C861410"
+		(property "LCSC" "C25819"
 			(at 208.28 180.34 0)
 			(hide yes)
@@
 					(reference "R87")
 					(unit 1))))
-		(property "Manufacturer" "Yageo"
+		(property "Manufacturer" "UNI-ROYAL(Uniroyal Elec)"
 			(at 208.28 180.34 0)
 			(hide yes)
@@
 				(font
 					(size 1.27 1.27))))
-		(property "Manufacturer Part" "RT0603BRD0744K2L"
+		(property "Manufacturer Part" "0603WAF4702T5E"
 			(at 208.28 180.34 0)
 			(hide yes)
@@
 				(font
 					(size 1.27 1.27))))
-		(property "LCSC Part" "C861410"
+		(property "LCSC Part" "C25819"
 			(at 208.28 180.34 0)
 			(hide yes)
@@
 					(size 1.27 1.27))
 				(justify left)))
-		(property "Value" "10k 0.1%"
+		(property "Value" "10k 1%"
 			(at 261.62 181.60999999999999 0)
 			(effects
@@
 					(size 1.27 1.27))
 				(justify left)))
-		(property "LCSC" "C95204"
+		(property "LCSC" "C25804"
 			(at 259.08 180.34 0)
 			(hide yes)
@@
 					(reference "R88")
 					(unit 1))))
-		(property "Manufacturer" "Yageo"
+		(property "Manufacturer" "UNI-ROYAL(Uniroyal Elec)"
 			(at 259.08 180.34 0)
 			(hide yes)
@@
 				(font
 					(size 1.27 1.27))))
-		(property "Manufacturer Part" "RT0603BRD0710KL"
+		(property "Manufacturer Part" "0603WAF1002T5E"
 			(at 259.08 180.34 0)
 			(hide yes)
@@
 				(font
 					(size 1.27 1.27))))
-		(property "LCSC Part" "C95204"
+		(property "LCSC Part" "C25804"
 			(at 259.08 180.34 0)
 			(hide yes)
@@
 					(size 1.27 1.27))
 				(justify left)))
-		(property "Value" "10k 0.1%"
+		(property "Value" "10k 1%"
 			(at 152.4 128.27 0)
 			(effects
@@
 					(size 1.27 1.27))
 				(justify left)))
-		(property "LCSC" "C95204"
+		(property "LCSC" "C25804"
 			(at 149.86 127 0)
 			(hide yes)
@@
 					(reference "R90")
 					(unit 1))))
-		(property "Manufacturer" "Yageo"
+		(property "Manufacturer" "UNI-ROYAL(Uniroyal Elec)"
 			(at 149.86 127 0)
 			(hide yes)
@@
 				(font
 					(size 1.27 1.27))))
-		(property "Manufacturer Part" "RT0603BRD0710KL"
+		(property "Manufacturer Part" "0603WAF1002T5E"
 			(at 149.86 127 0)
 			(hide yes)
@@
 				(font
 					(size 1.27 1.27))))
-		(property "LCSC Part" "C95204"
+		(property "LCSC Part" "C25804"
 			(at 149.86 127 0)
 			(hide yes)
@@
 					(size 1.27 1.27))
 				(justify left)))
-		(property "Value" "10k 0.1%"
+		(property "Value" "10k 1%"
 			(at 312.42 181.60999999999999 0)
 			(effects
@@
 					(size 1.27 1.27))
 				(justify left)))
-		(property "LCSC" "C95204"
+		(property "LCSC" "C25804"
 			(at 309.88 180.34 0)
 			(hide yes)
@@
 					(reference "R91")
 					(unit 1))))
-		(property "Manufacturer" "Yageo"
+		(property "Manufacturer" "UNI-ROYAL(Uniroyal Elec)"
 			(at 309.88 180.34 0)
 			(hide yes)
@@
 				(font
 					(size 1.27 1.27))))
-		(property "Manufacturer Part" "RT0603BRD0710KL"
+		(property "Manufacturer Part" "0603WAF1002T5E"
 			(at 309.88 180.34 0)
 			(hide yes)
@@
 				(font
 					(size 1.27 1.27))))
-		(property "LCSC Part" "C95204"
+		(property "LCSC Part" "C25804"
 			(at 309.88 180.34 0)
 			(hide yes)
