File: m3_design/assembly_review/logic_power_path.kicad_sch (KiCad schematic)
At the start: 16 parts, among them U10 TPS2553DBVR, U11 TPS2121RUXR

Commit message: Validate and harden R5 flight computer CAD
Parts:
- added C97, C98: 1uF 25V X7R 10%, rocket:C_0603_1608Metric, symbol M3:C
- added C99: 100nF 50V, rocket:C0402, symbol M3:C
- U10: Manufacturer (none) -> Texas Instruments; Manufacturer Part (none) -> TPS2553DBVR
- U11: Manufacturer (none) -> Texas Instruments; Manufacturer Part (none) -> TPS2121RUXR
Connections:
- net GND: now also C97.2, C98.2, C99.2
- net RAW_PROTECTED: now also C97.1
- net USB_LIMITED: now also C98.1
- net VLOGIC: now also C99.1
Changed lines of the file:
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@@
 	(title_block
 		(title "08 | USB limit, source mux and hold-up")
-		(date "2026-09-07")
-		(rev "M3-ASSY-R4")
+		(date "2026-10-12")
+		(rev "M3-ASSY-R5")
 		(company "Single-board M3 candidate; full system incomplete"))
 	(text "08 | USB limit, source mux and hold-up"
@@
 				(font
 					(size 1.27 1.27))))
+		(property "Manufacturer" "Texas Instruments"
+			(at 76.2 76.2 0)
+			(hide yes)
+			(effects
+				(font
+					(size 1.27 1.27))))
+		(property "Manufacturer Part" "TPS2553DBVR"
+			(at 76.2 76.2 0)
+			(hide yes)
+			(effects
+				(font
+					(size 1.27 1.27))))
 		(instances
 			(project "m3"
@@
 				(font
 					(size 1.27 1.27))))
+		(property "Manufacturer" "Texas Instruments"
+			(at 274.32 76.2 0)
+			(hide yes)
+			(effects
+				(font
+					(size 1.27 1.27))))
+		(property "Manufacturer Part" "TPS2121RUXR"
+			(at 274.32 76.2 0)
+			(hide yes)
+			(effects
+				(font
+					(size 1.27 1.27))))
 		(instances
 			(project "m3"
@@
 	(sheet_instances
 		(path "/"
-			(page "8"))))
+			(page "8")))
+	(symbol
+		(lib_id "M3:C")
+		(at 81.2800 152.4000 0)
+		(unit 1)
+		(in_bom yes)
+		(on_board yes)
+		(dnp no)
+		(property "Reference" "C97"
+			(at 83.8200 151.1300 0)
+			(effects
+				(font
+					(size 1.27 1.27))
+				(justify left)))
+		(property "Value" "1uF 25V X7R 10%"
+			(at 83.8200 153.6700 0)
+			(effects
+				(font
+					(size 1.27 1.27))
+				(justify left)))
+		(property "Footprint" "rocket:C_0603_1608Metric"
+			(at 81.2800 152.4000 0)
+			(hide yes)
+			(effects
+				(font
+					(size 1.27 1.27))
+				(justify left)))
+		(property "Datasheet" ""
+			(at 81.2800 152.4000 0)
+			(hide yes)
+			(effects
+				(font
+					(size 1.27 1.27))
+				(justify left)))
+		(property "LCSC" "C29936"
+			(at 81.2800 152.4000 0)
+			(hide yes)
+			(effects
+				(font
+					(size 1.27 1.27))
+				(justify left)))
+		(instances
+			(project "m3"
+				(path "/6007a7db-6a58-5660-8beb-956dea045ff8/98c21473-b271-5039-bfe5-b3672097f1da"
+					(reference "C97")
+					(unit 1))))
+		(property "Manufacturer" "Samsung Electro-Mechanics"
+			(at 81.2800 152.4000 0)
+			(hide yes)
+			(effects
+				(font
+					(size 1.27 1.27))))
+		(property "Manufacturer Part" "CL10B105KA8NNNC"
+			(at 81.2800 152.4000 0)
+			(hide yes)
+			(effects
+				(font
+					(size 1.27 1.27))))
+		(property "LCSC Part" "C29936"
+			(at 81.2800 152.4000 0)
+			(hide yes)
+			(effects
+				(font
+					(size 1.27 1.27)))))
+	(wire (pts (xy 81.28 148.5900) (xy 73.6600 148.5900)) (stroke (width 0) (type default)))
+	(global_label "RAW_PROTECTED" (shape passive) (at 73.6600 148.5900 0) (effects (font (size 1.05 1.05)) (justify right)))
+	(wire (pts (xy 81.28 156.2100) (xy 73.6600 156.2100)) (stroke (width 0) (type default)))
+	(global_label "GND" (shape passive) (at 73.6600 156.2100 0) (effects (font (size 1.05 1.05)) (justify right)))
+	(symbol
+		(lib_id "M3:C")
+		(at 152.4000 152.4000 0)
+		(unit 1)
+		(in_bom yes)
+		(on_board yes)
+		(dnp no)
+		(property "Reference" "C98"
+			(at 154.9400 151.1300 0)
+			(effects
+				(font
+					(size 1.27 1.27))
+				(justify left)))
+		(property "Value" "1uF 25V X7R 10%"
+			(at 154.9400 153.6700 0)
+			(effects
+				(font
+					(size 1.27 1.27))
+				(justify left)))
+		(property "Footprint" "rocket:C_0603_1608Metric"
+			(at 152.4000 152.4000 0)
+			(hide yes)
+			(effects
+				(font
+					(size 1.27 1.27))
+				(justify left)))
+		(property "Datasheet" ""
+			(at 152.4000 152.4000 0)
+			(hide yes)
+			(effects
+				(font
+					(size 1.27 1.27))
+				(justify left)))
+		(property "LCSC" "C29936"
+			(at 152.4000 152.4000 0)
+			(hide yes)
+			(effects
+				(font
+					(size 1.27 1.27))
+				(justify left)))
+		(instances
+			(project "m3"
+				(path "/6007a7db-6a58-5660-8beb-956dea045ff8/98c21473-b271-5039-bfe5-b3672097f1da"
+					(reference "C98")
+					(unit 1))))
+		(property "Manufacturer" "Samsung Electro-Mechanics"
+			(at 152.4000 152.4000 0)
+			(hide yes)
+			(effects
+				(font
+					(size 1.27 1.27))))
+		(property "Manufacturer Part" "CL10B105KA8NNNC"
+			(at 152.4000 152.4000 0)
+			(hide yes)
+			(effects
+				(font
+					(size 1.27 1.27))))
+		(property "LCSC Part" "C29936"
+			(at 152.4000 152.4000 0)
+			(hide yes)
+			(effects
+				(font
+					(size 1.27 1.27)))))
+	(wire (pts (xy 152.4 148.5900) (xy 144.7800 148.5900)) (stroke (width 0) (type default)))
+	(global_label "USB_LIMITED" (shape passive) (at 144.7800 148.5900 0) (effects (font (size 1.05 1.05)) (justify right)))
+	(wire (pts (xy 152.4 156.2100) (xy 144.7800 156.2100)) (stroke (width 0) (type default)))
+	(global_label "GND" (shape passive) (at 144.7800 156.2100 0) (effects (font (size 1.05 1.05)) (justify right)))
+	(symbol
+		(lib_id "M3:C")
+		(at 223.5200 152.4000 0)
+		(unit 1)
+		(in_bom yes)
+		(on_board yes)
+		(dnp no)
+		(property "Reference" "C99"
+			(at 226.0600 151.1300 0)
+			(effects
+				(font
+					(size 1.27 1.27))
+				(justify left)))
+		(property "Value" "100nF 50V"
+			(at 226.0600 153.6700 0)
+			(effects
+				(font
+					(size 1.27 1.27))
+				(justify left)))
+		(property "Footprint" "rocket:C0402"
+			(at 223.5200 152.4000 0)
+			(hide yes)
+			(effects
+				(font
+					(size 1.27 1.27))
+				(justify left)))
+		(property "Datasheet" ""
+			(at 223.5200 152.4000 0)
+			(hide yes)
+			(effects
+				(font
+					(size 1.27 1.27))
+				(justify left)))
+		(property "LCSC" "C307331"
+			(at 223.5200 152.4000 0)
+			(hide yes)
+			(effects
+				(font
+					(size 1.27 1.27))
+				(justify left)))
+		(property "Manufacturer" "Samsung Electro-Mechanics"
+			(at 223.5200 152.4000 0)
+			(hide yes)
+			(effects
+				(font
+					(size 1.27 1.27))
+				(justify left)))
+		(property "Manufacturer Part" "CL05B104KB54PNC"
+			(at 223.5200 152.4000 0)
+			(hide yes)
+			(effects
+				(font
+					(size 1.27 1.27))
+				(justify left)))
+		(instances
+			(project "m3"
+				(path "/6007a7db-6a58-5660-8beb-956dea045ff8/98c21473-b271-5039-bfe5-b3672097f1da"
+					(reference "C99")
+					(unit 1))))
+		(property "LCSC Part" "C307331"
+			(at 223.5200 152.4000 0)
+			(hide yes)
+			(effects
+				(font
+					(size 1.27 1.27)))))
+	(wire (pts (xy 223.52 148.5900) (xy 215.9000 148.5900)) (stroke (width 0) (type default)))
+	(global_label "VLOGIC" (shape passive) (at 215.9000 148.5900 0) (effects (font (size 1.05 1.05)) (justify right)))
+	(wire (pts (xy 223.52 156.2100) (xy 215.9000 156.2100)) (stroke (width 0) (type default)))
+	(global_label "GND" (shape passive) (at 215.9000 156.2100 0) (effects (font (size 1.05 1.05)) (justify right)))
+)
