File: m3_design/assembly_review/sensors.kicad_sch (KiCad schematic)
At the start: 12 parts, among them U3 W25Q128JVSIQ, U4 ICM-45686, U5 MS561101BA03

Commit message: M3-ASSY-R4: R3 validation fixes, new IMU, fault-tolerant pyro sensing
The board, schematic sheets and footprint library are generated from
R3 (533af8e) by m3_design/r4_build.sh (r4_lib.py, r4_sch.py,
r4_pcb.py). docs/REQUIREMENTS.md states what the board must do;
docs/M3_R4.md records every change, the thirteen evaluation passes
(twelve independent reviews) and the accepted deviations.

- IMU: ST LSM6DSV320X (16 g and 320 g, 4000 dps)
- Pyro: black ARM and orange igniter terminals, eight pyro spacing
  rules in m3.kicad_dru, sense dividers of 2 x 5.1k over 2 x 2k in
  parallel, 4.7k at each ADC pin (R168-R172)
- Pull-pin on a JST PH connector; JLC tooling holes
- Fab: Standard PCBA, 84 BOM lines, 205 placed parts, $80.12 per board
  at five boards (tools/jlc_cost.py); placement rotations verified
- Gate: tools/check.sh DRC 0, unconnected 0, schematic parity 0, ERC 0,
  audit OK; m3_design/check_actuators.py OK

Nothing has been built or measured, and there is no R4 firmware. The
open owner decisions and the bench tests are listed in STATUS.md.

Co-Authored-By: Claude Opus 5.5 <noreply@anthropic.com>
Parts:
- U4: value ICM-45686 -> LSM6DSV320X; LCSC C22459454 -> C26633007
- U5: Manufacturer (none) -> TE Connectivity; Manufacturer Part (none) -> MS561101BA03-50
Connections:
- net GND: no longer U4.10 (RESV_10), U4.11 (RESV_11)
- no-connect marks 1 -> 3
Other:
- note added: "Firmware: keep OIS_PU_DIS = 0 (pins 10/11 rely on the internal pull-ups); WHO_AM_I 0x73."
- note added: "U4 = ST LSM6DSV320X (R4): +/-16 g low-g + +/-32..320 g high-g accel, +/-4000 dps gyro, SPI <= 10 MHz. Pins 10/11 open per DS14623 table 2."
- note added: "U4: 4-wire SPI. INT2 open; OCS_aux/SDO_aux (pins 10/11) open, held by their internal pull-ups (DS14623 table 25)."
- note removed: "Firmware must disable the default pulls on tied auxiliary pads (DS-000577 section 4.1)."
- note removed: "U4: single-interface 4-wire SPI. Keep INT2 open; unused auxiliary pads grounded."
Changed lines of the file:
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@@
 		(title "03 | Memory and sensors")
 		(date "2026-09-07")
-		(rev "M3-ASSY-R3")
+		(rev "M3-ASSY-R4")
 		(company "Single-board M3 candidate; full system incomplete"))
 	(text "03 | Memory and sensors"
@@
 				(font
 					(size 1.27 1.27))))
-		(property "Value" "ICM-45686"
+		(property "Value" "LSM6DSV320X"
 			(at 200.66 67.31 0)
 			(effects
@@
 				(font
 					(size 1.27 1.27))))
-		(property "LCSC" "C22459454"
+		(property "LCSC" "C26633007"
 			(at 200.66 78.74 0)
 			(hide yes)
@@
 	(no_connect
 		(at 229.87 73.66)
-)
-	(wire
-		(pts
-			(xy 229.87 76.2)
-			(xy 234.95000000000002 76.2))
-		(stroke
-			(width 0)
-			(type default))
-)
-	(global_label "GND"
-		(shape passive)
-		(at 234.95000000000002 76.2 180)
-		(effects
-			(font
-				(size 1.05 1.05))
-			(justify left))
-)
-	(wire
-		(pts
-			(xy 229.87 78.74)
-			(xy 234.95000000000002 78.74))
-		(stroke
-			(width 0)
-			(type default))
-)
-	(global_label "GND"
-		(shape passive)
-		(at 234.95000000000002 78.74 180)
-		(effects
-			(font
-				(size 1.05 1.05))
-			(justify left))
 )
 	(wire
@@
 				(font
 					(size 1.27 1.27))))
+		(property "Manufacturer" "TE Connectivity"
+			(at 327.66 76.2 0)
+			(hide yes)
+			(effects
+				(font
+					(size 1.27 1.27))
+				(justify left)))
+		(property "Manufacturer Part" "MS561101BA03-50"
+			(at 327.66 76.2 0)
+			(hide yes)
+			(effects
+				(font
+					(size 1.27 1.27))
+				(justify left)))
 		(instances
 			(project "m3"
@@
 			(justify right))
 )
-	(text "U4: single-interface 4-wire SPI. Keep INT2 open; unused auxiliary pads grounded."
+	(text "U4: 4-wire SPI. INT2 open; OCS_aux/SDO_aux (pins 10/11) open, held by their internal pull-ups (DS14623 table 25)."
 		(at 20.32 205.74 0)
 		(effects
@@
 			(justify left))
 )
-	(text "Firmware must disable the default pulls on tied auxiliary pads (DS-000577 section 4.1)."
+	(text "Firmware: keep OIS_PU_DIS = 0 (pins 10/11 rely on the internal pull-ups); WHO_AM_I 0x73."
 		(at 20.32 213.36 0)
 		(effects
@@
 			(justify left))
 )
+	(no_connect
+		(at 229.87 76.2)
+)
+	(no_connect
+		(at 229.87 78.74)
+)
+	(text "U4 = ST LSM6DSV320X (R4): +/-16 g low-g + +/-32..320 g high-g accel, +/-4000 dps gyro, SPI <= 10 MHz. Pins 10/11 open per DS14623 table 2."
+		(at 20.32 260.35 0)
+		(effects
+			(font
+				(size 1.05 1.05))
+			(justify left))
+)
