File: m3_design/assembly_review/sensors.kicad_sch (KiCad schematic)
At the start: 12 parts, among them U3 W25Q128JVSIQ, U4 LSM6DSV320X, U5 MS561101BA03

Commit message: Validate and harden R5 flight computer CAD
Parts:
- C29, C30, C31, C32: Manufacturer (none) -> Samsung Electro-Mechanics; Manufacturer Part (none) -> CL05B104KO5NNNC
- R10, R11, R64: Manufacturer (none) -> UNI-ROYAL(Uniroyal Elec); Manufacturer Part (none) -> 0402WGF1002TCE
- R12, R13: Manufacturer (none) -> UNI-ROYAL(Uniroyal Elec); Manufacturer Part (none) -> 0402WGF4701TCE
- U4: Manufacturer (none) -> STMicroelectronics; Manufacturer Part (none) -> LSM6DSV320XTR
Changed lines of the file:
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@@
+				(font
+					(size 1.27 1.27))))
+		(property "Manufacturer" "STMicroelectronics"
+			(at 200.66 78.74 0)
+			(hide yes)
+			(effects
+				(font
+					(size 1.27 1.27))))
+		(property "Manufacturer Part" "LSM6DSV320XTR"
+			(at 200.66 78.74 0)
+			(hide yes)
+			(effects
 				(font
 					(size 1.27 1.27))))
@@
 					(size 1.27 1.27))
 				(justify left)))
+		(property "Manufacturer" "Samsung Electro-Mechanics"
+			(at 88.9 124.46 0)
+			(hide yes)
+			(effects
+				(font
+					(size 1.27 1.27))
+				(justify left)))
+		(property "Manufacturer Part" "CL05B104KO5NNNC"
+			(at 88.9 124.46 0)
+			(hide yes)
+			(effects
+				(font
+					(size 1.27 1.27))
+				(justify left)))
 		(instances
 			(project "m3"
@@
 					(size 1.27 1.27))
 				(justify left)))
+		(property "Manufacturer" "Samsung Electro-Mechanics"
+			(at 208.28 124.46 0)
+			(hide yes)
+			(effects
+				(font
+					(size 1.27 1.27))
+				(justify left)))
+		(property "Manufacturer Part" "CL05B104KO5NNNC"
+			(at 208.28 124.46 0)
+			(hide yes)
+			(effects
+				(font
+					(size 1.27 1.27))
+				(justify left)))
 		(instances
 			(project "m3"
@@
 					(size 1.27 1.27))
 				(justify left)))
+		(property "Manufacturer" "Samsung Electro-Mechanics"
+			(at 241.3 124.46 0)
+			(hide yes)
+			(effects
+				(font
+					(size 1.27 1.27))
+				(justify left)))
+		(property "Manufacturer Part" "CL05B104KO5NNNC"
+			(at 241.3 124.46 0)
+			(hide yes)
+			(effects
+				(font
+					(size 1.27 1.27))
+				(justify left)))
 		(instances
 			(project "m3"
@@
 					(size 1.27 1.27))
 				(justify left)))
+		(property "Manufacturer" "Samsung Electro-Mechanics"
+			(at 307.34 162.56 0)
+			(hide yes)
+			(effects
+				(font
+					(size 1.27 1.27))
+				(justify left)))
+		(property "Manufacturer Part" "CL05B104KO5NNNC"
+			(at 307.34 162.56 0)
+			(hide yes)
+			(effects
+				(font
+					(size 1.27 1.27))
+				(justify left)))
 		(instances
 			(project "m3"
@@
 					(size 1.27 1.27))
 				(justify left)))
+		(property "Manufacturer" "UNI-ROYAL(Uniroyal Elec)"
+			(at 43.18 124.46 0)
+			(hide yes)
+			(effects
+				(font
+					(size 1.27 1.27))
+				(justify left)))
+		(property "Manufacturer Part" "0402WGF1002TCE"
+			(at 43.18 124.46 0)
+			(hide yes)
+			(effects
+				(font
+					(size 1.27 1.27))
+				(justify left)))
 		(instances
 			(project "m3"
@@
 					(size 1.27 1.27))
 				(justify left)))
+		(property "Manufacturer" "UNI-ROYAL(Uniroyal Elec)"
+			(at 175.26 124.46 0)
+			(hide yes)
+			(effects
+				(font
+					(size 1.27 1.27))
+				(justify left)))
+		(property "Manufacturer Part" "0402WGF1002TCE"
+			(at 175.26 124.46 0)
+			(hide yes)
+			(effects
+				(font
+					(size 1.27 1.27))
+				(justify left)))
 		(instances
 			(project "m3"
@@
 					(size 1.27 1.27))
 				(justify left)))
+		(property "Manufacturer" "UNI-ROYAL(Uniroyal Elec)"
+			(at 307.34 124.46 0)
+			(hide yes)
+			(effects
+				(font
+					(size 1.27 1.27))
+				(justify left)))
+		(property "Manufacturer Part" "0402WGF4701TCE"
+			(at 307.34 124.46 0)
+			(hide yes)
+			(effects
+				(font
+					(size 1.27 1.27))
+				(justify left)))
 		(instances
 			(project "m3"
@@
 					(size 1.27 1.27))
 				(justify left)))
+		(property "Manufacturer" "UNI-ROYAL(Uniroyal Elec)"
+			(at 353.06 124.46 0)
+			(hide yes)
+			(effects
+				(font
+					(size 1.27 1.27))
+				(justify left)))
+		(property "Manufacturer Part" "0402WGF4701TCE"
+			(at 353.06 124.46 0)
+			(hide yes)
+			(effects
+				(font
+					(size 1.27 1.27))
+				(justify left)))
 		(instances
 			(project "m3"
@@
 			(at 353.06 162.56 0)
 			(hide yes)
+			(effects
+				(font
+					(size 1.27 1.27))
+				(justify left)))
+		(property "Manufacturer" "UNI-ROYAL(Uniroyal Elec)"
+			(at 353.06 162.56 0)
+			(hide yes)
+			(effects
+				(font
+					(size 1.27 1.27))
+				(justify left)))
+		(property "Manufacturer Part" "0402WGF1002TCE"
+			(at 353.06 162.56 0)
+			(hide yes)

Commit message: Complete R6 flight computer CAD and validated fabrication package
Add protected radio and GPS ports, reset-off port power, compact connectors and single-channel pyro layout. Close independent routing, ground-return and decoupling findings; record zero-error CAD checks and current manufacturing artifacts. Document 100 mm length, IMU stock hold and remaining firmware and hardware qualification.
Parts:
- C29, C30, C31, C32: value 100nF -> 100nF 50V X7R 10%; LCSC C1525 -> C307331; LCSC Part (none) -> C307331; Manufacturer Part CL05B104KO5NNNC -> CL05B104KB54PNC
Changed lines of the file:
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@@
 		(title "03 | Memory and sensors")
 		(date "2026-09-07")
-		(rev "M3-ASSY-R4")
+		(rev "M3-ASSY-R6")
 		(company "Single-board M3 candidate; full system incomplete"))
 	(text "03 | Memory and sensors"
@@
 					(size 1.27 1.27))
 				(justify left)))
-		(property "Value" "100nF"
+		(property "Value" "100nF 50V X7R 10%"
 			(at 91.44000000000001 125.73 0)
 			(effects
@@
 					(size 1.27 1.27))
 				(justify left)))
-		(property "LCSC" "C1525"
+		(property "LCSC" "C307331"
 			(at 88.9 124.46 0)
 			(hide yes)
@@
 					(size 1.27 1.27))
 				(justify left)))
-		(property "Manufacturer Part" "CL05B104KO5NNNC"
+		(property "Manufacturer Part" "CL05B104KB54PNC"
 			(at 88.9 124.46 0)
 			(hide yes)
@@
 				(path "/6007a7db-6a58-5660-8beb-956dea045ff8/3ba7ef49-2012-5f2a-98bd-e18f61ab4da0"
 					(reference "C29")
-					(unit 1)))))
+					(unit 1))))		(property "LCSC Part" "C307331"
+			(at 0 0 0)
+			(hide yes)
+			(effects
+				(font
+					(size 1.27 1.27))
+				(justify left)))
+)
 	(wire
 		(pts
@@
 					(size 1.27 1.27))
 				(justify left)))
-		(property "Value" "100nF"
+		(property "Value" "100nF 50V X7R 10%"
 			(at 210.82 125.73 0)
 			(effects
@@
 					(size 1.27 1.27))
 				(justify left)))
-		(property "LCSC" "C1525"
+		(property "LCSC" "C307331"
 			(at 208.28 124.46 0)
 			(hide yes)
@@
 					(size 1.27 1.27))
 				(justify left)))
-		(property "Manufacturer Part" "CL05B104KO5NNNC"
+		(property "Manufacturer Part" "CL05B104KB54PNC"
 			(at 208.28 124.46 0)
 			(hide yes)
@@
 				(path "/6007a7db-6a58-5660-8beb-956dea045ff8/3ba7ef49-2012-5f2a-98bd-e18f61ab4da0"
 					(reference "C30")
-					(unit 1)))))
+					(unit 1))))		(property "LCSC Part" "C307331"
+			(at 0 0 0)
+			(hide yes)
+			(effects
+				(font
+					(size 1.27 1.27))
+				(justify left)))
+)
 	(wire
 		(pts
@@
 					(size 1.27 1.27))
 				(justify left)))
-		(property "Value" "100nF"
+		(property "Value" "100nF 50V X7R 10%"
 			(at 243.84 125.73 0)
 			(effects
@@
 					(size 1.27 1.27))
 				(justify left)))
-		(property "LCSC" "C1525"
+		(property "LCSC" "C307331"
 			(at 241.3 124.46 0)
 			(hide yes)
@@
 					(size 1.27 1.27))
 				(justify left)))
-		(property "Manufacturer Part" "CL05B104KO5NNNC"
+		(property "Manufacturer Part" "CL05B104KB54PNC"
 			(at 241.3 124.46 0)
 			(hide yes)
@@
 				(path "/6007a7db-6a58-5660-8beb-956dea045ff8/3ba7ef49-2012-5f2a-98bd-e18f61ab4da0"
 					(reference "C31")
-					(unit 1)))))
+					(unit 1))))		(property "LCSC Part" "C307331"
+			(at 0 0 0)
+			(hide yes)
+			(effects
+				(font
+					(size 1.27 1.27))
+				(justify left)))
+)
 	(wire
 		(pts
@@
 					(size 1.27 1.27))
 				(justify left)))
-		(property "Value" "100nF"
+		(property "Value" "100nF 50V X7R 10%"
 			(at 309.88 163.82999999999998 0)
 			(effects
@@
 					(size 1.27 1.27))
 				(justify left)))
-		(property "LCSC" "C1525"
+		(property "LCSC" "C307331"
 			(at 307.34 162.56 0)
 			(hide yes)
@@
 					(size 1.27 1.27))
 				(justify left)))
-		(property "Manufacturer Part" "CL05B104KO5NNNC"
+		(property "Manufacturer Part" "CL05B104KB54PNC"
 			(at 307.34 162.56 0)
 			(hide yes)
@@
 				(path "/6007a7db-6a58-5660-8beb-956dea045ff8/3ba7ef49-2012-5f2a-98bd-e18f61ab4da0"
 					(reference "C32")
-					(unit 1)))))
-	(wire
-		(pts
+					(unit 1))))		(property "LCSC Part" "C307331"
+			(at 0 0 0)
+			(hide yes)
+			(effects
+				(font
+					(size 1.27 1.27))
+				(justify left)))
+)
+	(wire
+		(pts
