File: m3_design/assembly_review/mcu.kicad_sch (KiCad schematic)
At the start: 23 parts, among them J2 SWD 1x6, U1 STM32H743VIT6, Y1 25MHz CL8pF

Commit message: Validate and harden R5 flight computer CAD
Parts:
- C13, C14, C15, C16, C17, C18, C21, C24: Manufacturer (none) -> Samsung Electro-Mechanics; Manufacturer Part (none) -> CL05B104KO5NNNC
- C19, C20: Manufacturer (none) -> Samsung Electro-Mechanics; Manufacturer Part (none) -> CL10A225KO8NNNC
- C22: Manufacturer (none) -> Samsung Electro-Mechanics; Manufacturer Part (none) -> CL10A105KB8NNNC
- C23: Manufacturer (none) -> Samsung Electro-Mechanics; Manufacturer Part (none) -> CL10A475KO8NNNC
- C25, C26: Manufacturer (none) -> Samsung Electro-Mechanics; Manufacturer Part (none) -> CL05C100JB5NNNC
- R168, R169, R170, R171, R172: Manufacturer (none) -> UNI-ROYAL(Uniroyal Elec); Manufacturer Part (none) -> 0402WGF4701TCE
- R5: Manufacturer (none) -> UNI-ROYAL(Uniroyal Elec); Manufacturer Part (none) -> 0402WGF1002TCE
- U1: Manufacturer (none) -> STMicroelectronics; Manufacturer Part (none) -> STM32H743VIT6TR
- Y1: Manufacturer (none) -> NDK; Manufacturer Part (none) -> NX3225GA-25.000M-STD-CRG-2
