File: m3_design/assembly_review/mcu.kicad_sch (KiCad schematic)
At the start: 23 parts, among them J2 SWD 1x6, U1 STM32H743VIT6, Y1 25MHz CL8pF

Commit message: Complete R6 flight computer CAD and validated fabrication package
Add protected radio and GPS ports, reset-off port power, compact connectors and single-channel pyro layout. Close independent routing, ground-return and decoupling findings; record zero-error CAD checks and current manufacturing artifacts. Document 100 mm length, IMU stock hold and remaining firmware and hardware qualification.
Parts:
- removed R169, R171: 4.7k, rocket:R0402, symbol M3:R
- C13, C14, C15, C16, C17, C18, C21, C24: value 100nF -> 100nF 50V X7R 10%; LCSC C1525 -> C307331; LCSC Part (none) -> C307331; Manufacturer Part CL05B104KO5NNNC -> CL05B104KB54PNC
- J2: value SWD 1x6 -> TC2030-IDC-NL SWD; footprint rocket:HDR-TH_6P-P2.54-V-M-1x6 -> rocket:M3_TC2030_IDC_NL; LCSC C492405 -> (none); LCSC Part C492405 -> (none); Manufacturer XFCN -> Tag-Connect; Manufacturer Part PZ254V-11-06P -> TC2030-IDC-NL; now left out of the parts list
Connections:
- net 3V3: now also J2.1 (Pin_1); no longer J2.5 (Pin_5)
- net GND: now also J2.5 (Pin_5); no longer J2.1 (Pin_1)
- net IMU_INT1: now also U1.98 (PE1); no longer U1.40 (PE10)
- net NRST: now also J2.3 (Pin_3); no longer J2.4 (Pin_4)
- net SWCLK: now also J2.4 (Pin_4); no longer J2.2 (Pin_2)
- net SWDIO: now also J2.2 (Pin_2); no longer J2.3 (Pin_3)
- net TLM_FAULT_N: now reaches U1.31 (PA7)
- net TLM_PWR_EN: now reaches U1.51 (PB12)
- net RADIO_TX_MCU: now reaches U1.63 (PC6)
- net RADIO_RX_MCU: now reaches U1.64 (PC7)
- net RADIO_M0_MCU: now reaches U1.65 (PC8)
- net RADIO_M1_MCU: now reaches U1.66 (PC9)
- net RADIO_AUX_MCU: now reaches U1.67 (PA8)
- net GPS_TX_MCU: now reaches U1.68 (PA9)
- net GPS_RX_MCU: now reaches U1.69 (PA10)
- net ARM2_SENSE_MCU: no longer names the net of U1.32 (PC4)
- net PYRO2_CONT_MCU: no longer names the net of U1.16 (PC1)
- net PYRO2_GATE_N: no longer names the net of U1.4 (PE5)
- no-connect marks 37 -> 31
Other:
- note added: "CH1 sense: R168 4.7k -> PC0 continuity; R170 4.7k -> PC5 ARM; R172 4.7k -> PB0 RAW_ACT. Split divider safety retained. PE5/PC1/PC4 are now NC; PE3/PE6 remain sentinels. Never enable TRACE on PE2-PE6."
- note added: "IMU INT1: PE1 polled input only. EXTI1 remains PD1 power status. PE10 NC; pyro sentinels unchanged."
- note added: "J2 TC2030-IDC-NL: 1 VTref/3V3 | 2 SWDIO | 3 NRST | 4 SWCLK | 5 GND | 6 NC. BOOT0 remains at R5; use SWD or firmware jump for ROM boot."
- note added: "J2.1 is probe voltage reference only. Tag-Connect ARM20-CTX standard SWD mapping; pin 6 SWO is unused."
- note removed: "J2.5 is probe voltage reference. Do not connect a second power source."
- note removed: "J2: 1 GND | 2 SWCLK | 3 SWDIO | 4 NRST | 5 3V3 | 6 n/c (R4: BOOT0 stays on R5 at the MCU; DFU through SWD or a firmware jump to the system bootloader)"
- note removed: "R168-R172 (R4): 4.7k between each sense divider and its ADC pin: PYRO1/2_CONT -> PC0/PC1, ARM1/2_SENSE -> PC5/PC4, RAW_ACT_SENSE -> PB0. The dividers (2 x 5.1k in series over 2 x 2k in parallel, passes 11-12) keep each node <= 1.4 V (3.3 V at the 19.9 V clamp) with any one part shorted or open; these 4.7k limit the current only if two faults coincide (about 1 mA, Inference). ADC source 5.6 kohm (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"
