File: m3_design/assembly_review/mcu.kicad_sch (KiCad schematic)
At the start: 21 parts, among them J2 TC2030-IDC-NL SWD, U1 STM32H743VIT6, Y1 25MHz CL8pF

Commit message: M3-ASSY-R7: on-board GNSS and LoRa radio, clean-routing gate, owner-accepted deviations
R7 replaces R6's external radio/GPS harness ports with an on-board u-blox
MAX-F10S (U30, MAX-M10S drop-in) and EBYTE E22-900MM22S SX1262 radio (U31)
in an RF strip at the aft end, each with an edge-launch SMA jack (J30 GNSS,
J31 RADIO), RF ESD, an antenna-bias current limiter and DNP tuning pads.
The board grows to 46 x 118 mm (R6 copper translated +18 mm).

- Schematic, parts and footprints: r7_sch.py, r7_parts.py
- Reproducible board build from the SHA-checked R6 board: r7_build.sh
  (r7_pcb, r7_route, r7_redraw, r7_rework, r7_hygiene, r7_polish, r7_post)
- Gate: check_r7.py (RF contract), route_check.py (clean routing, M2)
  in tools/check.sh; fit_check, cost and procurement updated for R7
- Eight independent review passes with skeptic verification; pass 8 on
  this board found 0 Critical / 0 Major
- Owner accepted the deviation list on 2026-10-18 (R7_VALIDATION), with
  the 7.7 A servo-feed copper rise accepted as estimated

Board SHA-256 c872a3d30509cccf5f78b64cde48ef722ee85c7be23c4848b07ce4082a852de3.
tools/check.sh: DRC 0, unconnected 0, parity 0, ERC 0; audit, silk,
R7 contract, routing hygiene (0 failing), actuator contract and fit OK.
Before ordering: consign U4 and get JLC's forward-rail confirmation.

Co-Authored-By: Claude Opus 5.5 <noreply@anthropic.com>
Connections:
- net RADIO_RXEN: now reaches U1.45 (PE15)
- net RADIO_SCK_MCU: now reaches U1.52 (PB13)
- net RADIO_MISO_MCU: now reaches U1.53 (PB14)
- net RADIO_MOSI_MCU: now reaches U1.54 (PB15)
- net RADIO_BUSY: now reaches U1.55 (PD8)
- net RADIO_NRST: now reaches U1.56 (PD9)
- net RADIO_DIO1: now reaches U1.57 (PD10)
- net GNSS_TP_MCU: now reaches U1.61 (PD14)
- net GPS_RX_MCU: no longer names the net of U1.69 (PA10)
- net GPS_TX_MCU: no longer names the net of U1.68 (PA9)
- net RADIO_AUX_MCU: no longer names the net of U1.67 (PA8)
- net RADIO_M0_MCU renamed GNSS_RESET_N
- net RADIO_M1_MCU: no longer names the net of U1.66 (PC9)
- net RADIO_RX_MCU renamed GNSS_TXD_MCU
- net RADIO_TX_MCU renamed GNSS_RXD_MCU
- net TLM_FAULT_N: no longer names the net of U1.31 (PA7)
- net TLM_PWR_EN renamed RADIO_NSS
- no-connect marks 31 -> 28
Other:
- note added: "R7 (sheet 15): radio SPI2 PB12 NSS, PB13 SCK, PB14 MISO, PB15 MOSI; PD8 BUSY, PD9 NRST, PD10 DIO1, PE15 RXEN. GNSS USART6 PC6/PC7, PC8 RESET_N (open drain), PD14 TIMEPULSE. PA7, PC9, PA8, PA9, PA10 NC."
Changed lines of the file:
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@@
 		(title "02 | MCU, clock and debug")
 		(date "2026-09-07")
-		(rev "M3-ASSY-R6")
+		(rev "M3-ASSY-R7")
 		(company "Single-board M3 candidate; full system incomplete"))
 	(text "02 | MCU, clock and debug"
@@
 )
 	(no_connect
-		(at 119.38 130.81)
-)
-	(no_connect
-		(at 119.38 135.89)
-)
-	(no_connect
-		(at 119.38 138.43)
-)
-	(no_connect
-		(at 119.38 140.97)
-)
-	(no_connect
-		(at 119.38 143.51)
-)
-	(no_connect
-		(at 119.38 146.05)
-)
-	(no_connect
-		(at 119.38 148.59)
-)
-	(no_connect
-		(at 119.38 151.13)
-)
-	(no_connect
 		(at 119.38 166.37)
 )
@@
 			(justify left))
 )
+	(no_connect
+		(at 119.38 69.85)
+)
+	(no_connect
+		(at 119.38 82.55)
+)
+	(no_connect
+		(at 119.38 105.41)
+)
 	(wire
 		(pts
-			(xy 63.5 140.97)
-			(xy 58.42 140.97))
+			(xy 325.12 58.42)
+			(xy 320.04 58.42))
 		(stroke
 			(width 0)
 			(type default))
 )
-	(global_label "RADIO_TX_MCU"
+	(global_label "3V3"
 		(shape passive)
-		(at 58.42 140.97 0)
+		(at 320.04 58.42 0)
 		(effects
 			(font
@@
 	(wire
 		(pts
-			(xy 63.5 143.51)
-			(xy 58.42 143.51))
+			(xy 325.12 60.96)
+			(xy 320.04 60.96))
 		(stroke
 			(width 0)
 			(type default))
 )
-	(global_label "RADIO_RX_MCU"
+	(global_label "SWDIO"
 		(shape passive)
-		(at 58.42 143.51 0)
+		(at 320.04 60.96 0)
 		(effects
 			(font
@@
 	(wire
 		(pts
-			(xy 119.38 153.67)
-			(xy 124.46 153.67))
+			(xy 325.12 63.5)
+			(xy 320.04 63.5))
 		(stroke
 			(width 0)
 			(type default))
 )
-	(global_label "RADIO_M0_MCU"
+	(global_label "NRST"
 		(shape passive)
-		(at 124.46 153.67 180)
+		(at 320.04 63.5 0)
 		(effects
 			(font
 				(size 1.05 1.05))
-			(justify left))
+			(justify right))
 )
 	(wire
 		(pts
-			(xy 119.38 156.21)
-			(xy 124.46 156.21))
+			(xy 325.12 66.04)
+			(xy 320.04 66.04))
 		(stroke
 			(width 0)
 			(type default))
 )
-	(global_label "RADIO_M1_MCU"
+	(global_label "SWCLK"
 		(shape passive)
-		(at 124.46 156.21 180)
+		(at 320.04 66.04 0)
 		(effects
 			(font
 				(size 1.05 1.05))
-			(justify left))
+			(justify right))
 )
 	(wire
 		(pts
-			(xy 119.38 158.75)
-			(xy 124.46 158.75))
+			(xy 325.12 68.58)
+			(xy 320.04 68.58))
 		(stroke
 			(width 0)
 			(type default))
 )
-	(global_label "RADIO_AUX_MCU"
+	(global_label "GND"
 		(shape passive)
-		(at 124.46 158.75 180)
+		(at 320.04 68.58 0)
 		(effects
 			(font
 				(size 1.05 1.05))
-			(justify left))
+			(justify right))
+)
+	(no_connect
+		(at 325.12 71.12)
+)
+	(no_connect
+		(at 119.38 191.77)
+)
+	(no_connect
+		(at 63.5 115.57)
 )
 	(wire
 		(pts
-			(xy 119.38 161.29)
-			(xy 124.46 161.29))
+			(xy 119.38 194.31)
+			(xy 124.46 194.31))
 		(stroke
 			(width 0)
 			(type default))
 )
-	(global_label "GPS_TX_MCU"
+	(global_label "IMU_INT1"
 		(shape passive)
-		(at 124.46 161.29 180)
+		(at 124.46 194.31 180)
+		(effects
+			(font
+				(size 1.05 1.05))
+			(justify left))
+)
+	(text "IMU INT1: PE1 polled input only. EXTI1 remains PD1 power status. PE10 NC; pyro sentinels unchanged."
+		(at 40.64 248.92 0)
 		(effects
 			(font
@@
 	(wire
 		(pts
-			(xy 119.38 163.83)
-			(xy 124.46 163.83))
+			(xy 119.38 130.81)
+			(xy 124.46 130.81))
 		(stroke
 			(width 0)
 			(type default))
 )
-	(global_label "GPS_RX_MCU"
+	(global_label "RADIO_RXEN"
 		(shape passive)
-		(at 124.46 163.83 180)
+		(at 124.46 130.81 180)
 		(effects
 			(font
@@
 			(justify left))
 )
-	(no_connect
-		(at 119.38 69.85)
-)
-	(no_connect
-		(at 119.38 82.55)
+	(wire
+		(pts
+			(xy 119.38 133.35)
+			(xy 124.46 133.35))
+		(stroke
+			(width 0)
+			(type default))
 )
-	(no_connect
-		(at 119.38 105.41)
+	(global_label "RADIO_NSS"
+		(shape passive)
+		(at 124.46 133.35 180)
+		(effects
+			(font
+				(size 1.05 1.05))
+			(justify left))
 )
 	(wire
 		(pts
-			(xy 325.12 58.42)
-			(xy 320.04 58.42))
+			(xy 119.38 135.89)
+			(xy 124.46 135.89))
 		(stroke
 			(width 0)
 			(type default))
 )
-	(global_label "3V3"
+	(global_label "RADIO_SCK_MCU"
 		(shape passive)
-		(at 320.04 58.42 0)
+		(at 124.46 135.89 180)
 		(effects
 			(font
 				(size 1.05 1.05))
-			(justify right))
+			(justify left))
 )
 	(wire
 		(pts
-			(xy 325.12 60.96)
-			(xy 320.04 60.96))
+			(xy 119.38 138.43)
+			(xy 124.46 138.43))
 		(stroke
 			(width 0)
 			(type default))
 )
-	(global_label "SWDIO"
+	(global_label "RADIO_MISO_MCU"
 		(shape passive)
-		(at 320.04 60.96 0)
+		(at 124.46 138.43 180)
 		(effects
 			(font
 				(size 1.05 1.05))
-			(justify right))
+			(justify left))
 )
 	(wire
 		(pts
-			(xy 325.12 63.5)
-			(xy 320.04 63.5))
+			(xy 119.38 140.97)
+			(xy 124.46 140.97))
 		(stroke
 			(width 0)
 			(type default))
 )
-	(global_label "NRST"
+	(global_label "RADIO_MOSI_MCU"
 		(shape passive)
-		(at 320.04 63.5 0)
+		(at 124.46 140.97 180)
 		(effects
 			(font
 				(size 1.05 1.05))
-			(justify right))
+			(justify left))
 )
 	(wire
 		(pts
-			(xy 325.12 66.04)
-			(xy 320.04 66.04))
+			(xy 119.38 143.51)
+			(xy 124.46 143.51))
 		(stroke
 			(width 0)
 			(type default))
 )
-	(global_label "SWCLK"
+	(global_label "RADIO_BUSY"
 		(shape passive)
-		(at 320.04 66.04 0)
+		(at 124.46 143.51 180)
 		(effects
 			(font
 				(size 1.05 1.05))
-			(justify right))
+			(justify left))
 )
 	(wire
 		(pts
-			(xy 325.12 68.58)
-			(xy 320.04 68.58))
+			(xy 119.38 146.05)
+			(xy 124.46 146.05))
 		(stroke
 			(width 0)
 			(type default))
 )
-	(global_label "GND"
+	(global_label "RADIO_NRST"
 		(shape passive)
-		(at 320.04 68.58 0)
+		(at 124.46 146.05 180)
 		(effects
 			(font
 				(size 1.05 1.05))
-			(justify right))
-)
-	(no_connect
-		(at 325.12 71.12)
+			(justify left))
 )
 	(wire
 		(pts
-			(xy 119.38 133.35)
-			(xy 124.46 133.35))
+			(xy 119.38 148.59)
+			(xy 124.46 148.59))
 		(stroke
 			(width 0)
 			(type default))
 )
-	(global_label "TLM_PWR_EN"
+	(global_label "RADIO_DIO1"
 		(shape passive)
-		(at 124.46 133.35 180)
+		(at 124.46 148.59 180)
 		(effects
 			(font
@@
 			(justify left))
 )
-	(no_connect
-		(at 119.38 191.77)
-)
 	(wire
 		(pts
-			(xy 119.38 102.87)
-			(xy 124.46 102.87))
+			(xy 119.38 151.13)
+			(xy 124.46 151.13))
 		(stroke
 			(width 0)
 			(type default))
 )
-	(global_label "TLM_FAULT_N"
+	(global_label "GNSS_TP_MCU"
 		(shape passive)
-		(at 124.46 102.87 180)
+		(at 124.46 151.13 180)
 		(effects
 			(font
@@
 			(justify left))
 )
-	(no_connect
-		(at 63.5 115.57)
+	(wire
+		(pts
+			(xy 63.5 140.97)
+			(xy 58.42 140.97))
+		(stroke
+			(width 0)
+			(type default))
+)
+	(global_label "GNSS_RXD_MCU"
+		(shape passive)
+		(at 58.42 140.97 0)
+		(effects
+			(font
+				(size 1.05 1.05))
+			(justify right))
 )
 	(wire
 		(pts
-			(xy 119.38 194.31)
-			(xy 124.46 194.31))
+			(xy 63.5 143.51)
+			(xy 58.42 143.51))
 		(stroke
 			(width 0)
 			(type default))
 )
-	(global_label "IMU_INT1"
+	(global_label "GNSS_TXD_MCU"
 		(shape passive)
-		(at 124.46 194.31 180)
+		(at 58.42 143.51 0)
+		(effects
+			(font
+				(size 1.05 1.05))
+			(justify right))
+)
+	(wire
+		(pts
+			(xy 119.38 153.67)
+			(xy 124.46 153.67))
+		(stroke
+			(width 0)
+			(type default))
+)
+	(global_label "GNSS_RESET_N"
+		(shape passive)
+		(at 124.46 153.67 180)
 		(effects
 			(font
@@
 			(justify left))
 )
-	(text "IMU INT1: PE1 polled input only. EXTI1 remains PD1 power status. PE10 NC; pyro sentinels unchanged."
-		(at 40.64 248.92 0)
+	(no_connect
+		(at 119.38 102.87)
+)
+	(no_connect
+		(at 119.38 156.21)
+)
+	(no_connect
+		(at 119.38 158.75)
+)
+	(no_connect
+		(at 119.38 161.29)
+)
+	(no_connect
+		(at 119.38 163.83)
+)
+	(text "R7 (sheet 15): radio SPI2 PB12 NSS, PB13 SCK, PB14 MISO, PB15 MOSI; PD8 BUSY, PD9 NRST, PD10 DIO1, PE15 RXEN. GNSS USART6 PC6/PC7, PC8 RESET_N (open drain), PD14 TIMEPULSE. PA7, PC9, PA8, PA9, PA10 NC."
+		(at 20.32 259.08 0)
 		(effects
 			(font

Commit message: M3-ASSY-R8: re-placed layout with planned-bus routing, owner-accepted deviations
R8 keeps R7's circuit, RF strip and CH1 pyro block (copied rigidly and
hash-asserted) and re-places everything else: U1 rotated so its free
pins face the RF strip, each block beside the U1 face it talks to, input
protection back at J1, and a fresh deterministic build (r8_build.sh)
with planned-bus routing, no autorouter and no patch stages.

Against R7: signal track 3.36 m -> 1.50 m, signal vias 217 -> 55,
simplicity index 100 -> 15.3, gate exceptions 74 -> 3, hard routing-rule
instances 10 -> 1, 7.7 A neck rise 38/30/44 -> 17.6/14.8/22.3 C,
unreferenced critical samples 27.9 % -> 11.1 %, non-pyro nets within
3 mm of armed copper 23 -> 7.

- Gate: check_r8 (pin contract from pin_table.tsv, F10 separation,
  battery/pyro clearance, loader-pin rule, rigid hashes), route_check
  profile r8, scorecard, dc_solve --necks, reference_audit, paste_check
- Review: passes 2, 3 and 4 found 0 Critical / 0 Major in all eight
  dimensions; pass 5 re-checked the final board (routing, planes,
  integrity) with 0 Critical / 0 Major
- Owner accepted the R8 deviation list on 2026-10-20, including the C10
  vibration item and the listed agent decisions

Board SHA-256 cc044ea0922ff826df19af9d9726d92c096ab2b127025b55d123d8772e5fb4a7.
tools/check.sh: DRC 0, unconnected 0, parity 0, ERC 0; audit, silk,
R8 contract, routing hygiene (0 failing, 3 allowlisted), actuator
contract and fit OK. Before ordering: consign U4, JLC tab acceptance,
cost/stock run within 24 h.

Co-Authored-By: Claude Opus 5.5 <noreply@anthropic.com>
Connections:
- net BAT_FAULT_N: now also U1.28 (PA4); no longer U1.81 (PD0)
- net BUZZ_DRV: now also U1.7 (PC13); no longer U1.29 (PA5)
- net CAM_FAULT_N: now also U1.41 (PE11); no longer U1.85 (PD4)
- net CAM_MCU_RX: now also U1.37 (PE7); no longer U1.47 (PB11)
- net CAM_MCU_TX: now also U1.38 (PE8); no longer U1.46 (PB10)
- net CAM_PWR_EN: now also U1.42 (PE12); no longer U1.84 (PD3)
- net CAM_UART_OE: now also U1.31 (PA7); no longer U1.7 (PC13)
- net GNSS_RESET_N: now also U1.61 (PD14); no longer U1.65 (PC8)
- net GNSS_TP_MCU: now also U1.62 (PD15); no longer U1.61 (PD14)
- net LED_RED: now also U1.86 (PD5); no longer U1.38 (PE8)
- net LED_YEL: now also U1.88 (PD7); no longer U1.37 (PE7)
- net LOGIC_SOURCE_ST: now also U1.29 (PA5); no longer U1.82 (PD1)
- net RADIO_DIO1: now also U1.45 (PE15); no longer U1.57 (PD10)
- net RADIO_MISO_MCU: now also U1.54 (PB15); no longer U1.53 (PB14)
- net RADIO_MOSI_MCU: now also U1.53 (PB14); no longer U1.54 (PB15)
- net RADIO_NRST: now also U1.39 (PE9); no longer U1.56 (PD9)
- net RADIO_NSS: now also U1.47 (PB11); no longer U1.51 (PB12)
- net RADIO_RXEN: now also U1.56 (PD9); no longer U1.45 (PE15)
- net RADIO_SCK_MCU: now also U1.46 (PB10); no longer U1.52 (PB13)
- net VBUS_SENSE: now also U1.65 (PC8); no longer U1.62 (PD15)
Other:
- note added: "IMU INT1: PE1 polled input only. R8 EXTI: 4 BAT_FAULT_N PA4, 5 LOGIC_SOURCE_ST PA5, 6 USB_FAULT_N PD6, 8 VBUS_SENSE PC8, 11 CAM_FAULT_N PE11, 14 PULLPIN PC14, 15 RADIO_DIO1 PE15. PE10 NC; pyro sentinels unchanged."
- note added: "Pins the ROM bootloader drives (AN2606 Table 135; D5) carry only SERVO3 PA2, RADIO_SCK PB10, RADIO_MOSI PB14, USB PA11/PA12, QSPI_NCS PB6 and I2C1_SDA PB9; PA6, PA8, PA9, PA10, PC9, PC11, PE13 stay NC."
- note added: "R2: PE3 (pin 2) and PE6 (pin 5) are pyro-gate sentinels - no net, firmware drives them low. R8: LED_RED on PD5 (pin 86), LED_YEL on PD7 (pin 88)."
- note added: "R8 (sheet 15): radio SPI2 PB10 SCK, PB11 NSS (software; R310 100k to 3V3), PB14 MOSI / PB15 MISO (AF5 with SPI_CFG2.IOSWP = 1); PD8 BUSY (polled), PD9 RXEN, PE9 NRST, PE15 DIO1. GNSS USART6 PC6/PC7, PD14 RESET_N (open drain), PD15 TIMEPULSE (TIM4_CH4)."
- note added: "R8 follow-on moves (D3): BUZZ_DRV PC13, BAT_FAULT_N PA4, LOGIC_SOURCE_ST PA5, CAM_UART_OE PA7, camera UART7 PE7 RX / PE8 TX, CAM_FAULT_N PE11, CAM_PWR_EN PE12, VBUS_SENSE PC8, LEDs PD5 / PD7. Freed, NC: PB12, PB13, PD10, PD0, PD1, PD3, PD4."
- note added: "R8: camera enable CAM_PWR_EN on PE12 / pin42, fault input CAM_FAULT_N on PE11 / pin41 (GPIO only, SPI4 never enabled); no actuation changes."
- note removed: "Added PD3 / pin84: camera enable. PD4 / pin85: fault input; no actuation changes."
- note removed: "IMU INT1: PE1 polled input only. EXTI1 remains PD1 power status. PE10 NC; pyro sentinels unchanged."
- note removed: "R2: PE3 (pin 2) and PE6 (pin 5) are pyro-gate sentinels - no net, firmware drives them low. LED_RED moved to PE8."
- note removed: "R7 (sheet 15): radio SPI2 PB12 NSS, PB13 SCK, PB14 MISO, PB15 MOSI; PD8 BUSY, PD9 NRST, PD10 DIO1, PE15 RXEN. GNSS USART6 PC6/PC7, PC8 RESET_N (open drain), PD14 TIMEPULSE. PA7, PC9, PA8, PA9, PA10 NC."
