File: m3_design/assembly_review/mcu.kicad_sch (KiCad schematic)
At the start: 21 parts, among them J2 TC2030-IDC-NL SWD, U1 STM32H743VIT6, Y1 25MHz CL8pF

Commit message: R10: m3_design/r10_build.sh and per-family stage gate; m3_design/assembly_review rebuilt as M3-ASSY-R10 (board 883d2db5..., 46 x 90 mm); tools/check.sh passes at zero; binding note bound to the board
Co-Authored-By: Claude Opus 5.5 <noreply@anthropic.com>
Connections:
- net RADIO_NRST is gone; now on net CAM_UART_OE: U1.39 (PE9)
- net BAT_FAULT_N: now also U1.29 (PA5); no longer U1.28 (PA4)
- net BUZZ_DRV: now also U1.8 (PC14); no longer U1.7 (PC13)
- net CAM_FAULT_N: now also U1.42 (PE12); no longer U1.41 (PE11)
- net CAM_PWR_EN: now also U1.41 (PE11); no longer U1.42 (PE12)
- net CAM_UART_OE: no longer U1.31 (PA7)
- net LOGIC_SOURCE_ST: now also U1.28 (PA4); no longer U1.29 (PA5)
- net PULLPIN: now also U1.7 (PC13); no longer U1.8 (PC14)
- net VLOGIC_SENSE: now also U1.30 (PA6); no longer U1.17 (PC2_C)
- net RADIO_RX_MCU: now reaches U1.51 (PB12)
- net RADIO_TX_MCU: now reaches U1.52 (PB13)
- net GPS_FAULT_N: now reaches U1.57 (PD10)
- net GNSS_RESET_N renamed GPS_PWR_EN
- net GNSS_RXD_MCU renamed GPS_TX_MCU
- net GNSS_TP_MCU renamed GPS_UART_OE
- net GNSS_TXD_MCU renamed GPS_RX_MCU
- net RADIO_BUSY renamed RADIO_PWR_EN
- net RADIO_DIO1 renamed RADIO_UART_OE
- net RADIO_MISO_MCU: no longer names the net of U1.54 (PB15)
- net RADIO_MOSI_MCU: no longer names the net of U1.53 (PB14)
- net RADIO_NSS: no longer names the net of U1.47 (PB11)
- net RADIO_RXEN renamed RADIO_FAULT_N
- net RADIO_SCK_MCU: no longer names the net of U1.46 (PB10)
- no-connect marks 28 -> 30
Other:
- note added: "R10: USART6 PC6/PC7 AF7 GPS; UART5 PB13/PB12 AF14 radio. Port EN and OE default low. EXTI10 GPS_FAULT_N; EXTI9 RADIO_FAULT_N; EXTI12 CAM_FAULT_N; EXTI4 LOGIC_SOURCE_ST (PA4), EXTI5 BAT_FAULT_N (PA5); VLOGIC_SENSE ADC on PA6 (D-R2-09). PE1 remains polled."
- note removed: "IMU INT1: PE1 polled input only. R8 EXTI: 4 BAT_FAULT_N PA4, 5 LOGIC_SOURCE_ST PA5, 6 USB_FAULT_N PD6, 8 VBUS_SENSE PC8, 11 CAM_FAULT_N PE11, 14 PULLPIN PC14, 15 RADIO_DIO1 PE15. PE10 NC; pyro sentinels unchanged."
- note removed: "R8 (sheet 15): radio SPI2 PB10 SCK, PB11 NSS (software; R310 100k to 3V3), PB14 MOSI / PB15 MISO (AF5 with SPI_CFG2.IOSWP = 1); PD8 BUSY (polled), PD9 RXEN, PE9 NRST, PE15 DIO1. GNSS USART6 PC6/PC7, PD14 RESET_N (open drain), PD15 TIMEPULSE (TIM4_CH4)."
Changed lines of the file:
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@@
 		(title "02 | MCU, clock and debug")
 		(date "2026-09-07")
-		(rev "M3-ASSY-R9")
+		(rev "M3-ASSY-R10")
 		(company "Single-board M3 candidate; full system incomplete"))
 	(text "02 | MCU, clock and debug"
@@
 			(type default))
 )
-	(global_label "BUZZ_DRV"
+	(global_label "PULLPIN"
 		(shape passive)
 		(at 58.42 77.47 0)
@@
 	(wire
 		(pts
-			(xy 63.5 92.71)
-			(xy 58.42 92.71))
-		(stroke
-			(width 0)
-			(type default))
-)
-	(global_label "VLOGIC_SENSE"
-		(shape passive)
-		(at 58.42 92.71 0)
-		(effects
-			(font
-				(size 1.05 1.05))
-			(justify right))
-)
-	(wire
-		(pts
 			(xy 63.5 95.25)
 			(xy 58.42 95.25))
@@
 	(wire
 		(pts
-			(xy 63.5 118.11)
-			(xy 58.42 118.11))
-		(stroke
-			(width 0)
-			(type default))
-)
-	(global_label "RADIO_SCK_MCU"
-		(shape passive)
-		(at 58.42 118.11 0)
-		(effects
-			(font
-				(size 1.05 1.05))
-			(justify right))
-)
-	(wire
-		(pts
-			(xy 63.5 120.65)
-			(xy 58.42 120.65))
-		(stroke
-			(width 0)
-			(type default))
-)
-	(global_label "RADIO_NSS"
-		(shape passive)
-		(at 58.42 120.65 0)
-		(effects
-			(font
-				(size 1.05 1.05))
-			(justify right))
-)
-	(wire
-		(pts
 			(xy 63.5 123.19)
 			(xy 58.42 123.19))
@@
 			(type default))
 )
-	(global_label "GNSS_TP_MCU"
+	(global_label "GPS_UART_OE"
 		(shape passive)
 		(at 58.42 138.43 0)
@@
 )
 	(no_connect
-		(at 119.38 100.33)
-)
-	(no_connect
 		(at 119.38 125.73)
 )
@@
 			(type default))
 )
-	(global_label "LOGIC_SOURCE_ST"
+	(global_label "BAT_FAULT_N"
 		(shape input)
 		(at 127 97.79 0)
@@
 			(type default))
 )
-	(global_label "PULLPIN"
+	(global_label "BUZZ_DRV"
 		(shape passive)
 		(at 127 74.93 0)
@@
 			(justify left))
 )
-	(text "IMU INT1: PE1 polled input only. R8 EXTI: 4 BAT_FAULT_N PA4, 5 LOGIC_SOURCE_ST PA5, 6 USB_FAULT_N PD6, 8 VBUS_SENSE PC8, 11 CAM_FAULT_N PE11, 14 PULLPIN PC14, 15 RADIO_DIO1 PE15. PE10 NC; pyro sentinels unchanged."
-		(at 40.64 248.92 0)
-		(effects
-			(font
-				(size 1.05 1.05))
-			(justify left))
-)
 	(wire
 		(pts
@@
 			(type default))
 )
-	(global_label "RADIO_DIO1"
+	(global_label "RADIO_UART_OE"
 		(shape passive)
 		(at 124.46 130.81 180)
@@
 	(wire
 		(pts
-			(xy 119.38 138.43)
-			(xy 124.46 138.43))
-		(stroke
-			(width 0)
-			(type default))
-)
-	(global_label "RADIO_MOSI_MCU"
-		(shape passive)
-		(at 124.46 138.43 180)
-		(effects
-			(font
-				(size 1.05 1.05))
-			(justify left))
-)
-	(wire
-		(pts
-			(xy 119.38 140.97)
-			(xy 124.46 140.97))
-		(stroke
-			(width 0)
-			(type default))
-)
-	(global_label "RADIO_MISO_MCU"
-		(shape passive)
-		(at 124.46 140.97 180)
-		(effects
-			(font
-				(size 1.05 1.05))
-			(justify left))
-)
-	(wire
-		(pts
 			(xy 119.38 143.51)
 			(xy 124.46 143.51))
@@
 			(type default))
 )
-	(global_label "RADIO_BUSY"
+	(global_label "RADIO_PWR_EN"
 		(shape passive)
 		(at 124.46 143.51 180)
@@
 			(type default))
 )
-	(global_label "RADIO_RXEN"
+	(global_label "RADIO_FAULT_N"
 		(shape passive)
 		(at 124.46 146.05 180)
@@
 			(type default))
 )
-	(global_label "GNSS_RESET_N"
+	(global_label "GPS_PWR_EN"
 		(shape passive)
 		(at 124.46 151.13 180)
@@
 			(type default))
 )
-	(global_label "GNSS_RXD_MCU"
+	(global_label "GPS_TX_MCU"
 		(shape passive)
 		(at 58.42 140.97 0)
@@
 			(type default))
 )
-	(global_label "GNSS_TXD_MCU"
+	(global_label "GPS_RX_MCU"
 		(shape passive)
 		(at 58.42 143.51 0)
@@
 		(at 119.38 163.83)
 )
-	(text "R8 (sheet 15): radio SPI2 PB10 SCK, PB11 NSS (software; R310 100k to 3V3), PB14 MOSI / PB15 MISO (AF5 with SPI_CFG2.IOSWP = 1); PD8 BUSY (polled), PD9 RXEN, PE9 NRST, PE15 DIO1. GNSS USART6 PC6/PC7, PD14 RESET_N (open drain), PD15 TIMEPULSE (TIM4_CH4)."
-		(at 20.32 259.08 0)
-		(effects
-			(font
-				(size 1.05 1.05))
-			(justify left))
-)
 	(wire
 		(pts
@@
 			(type default))
 )
-	(global_label "BAT_FAULT_N"
+	(global_label "LOGIC_SOURCE_ST"
 		(shape input)
 		(at 124.46 95.25 180)
@@
 	(wire
 		(pts
-			(xy 119.38 102.87)
-			(xy 124.46 102.87))
-		(stroke
-			(width 0)
-			(type default))
-)
-	(global_label "CAM_UART_OE"
-		(shape passive)
-		(at 124.46 102.87 180)
-		(effects
-			(font
-				(size 1.05 1.05))
-			(justify left))
-)
-	(wire
-		(pts
 			(xy 119.38 118.11)
 			(xy 124.46 118.11))
@@
 			(type default))
 )
-	(global_label "RADIO_NRST"
+	(global_label "CAM_UART_OE"
 		(shape passive)
 		(at 124.46 118.11 180)
@@
 			(type default))
 )
-	(global_label "CAM_FAULT_N"
+	(global_label "CAM_PWR_EN"
 		(shape passive)
 		(at 124.46 120.65 180)
@@
 			(type default))
 )
-	(global_label "CAM_PWR_EN"
+	(global_label "CAM_FAULT_N"
 		(shape passive)
 		(at 124.46 123.19 180)
@@
 )
 	(no_connect
-		(at 119.38 133.35)
-)
-	(no_connect
-		(at 119.38 135.89)
-)
-	(no_connect
-		(at 119.38 148.59)
-)
-	(no_connect
 		(at 119.38 176.53)
 )
@@
 		(effects
 			(font
+				(size 1.05 1.05))
+			(justify left))
+)
+	(no_connect
+		(at 63.5 92.71)
+)
+	(wire
+		(pts
+			(xy 119.38 100.33)
+			(xy 124.46 100.33))
+		(stroke
+			(width 0)
+			(type default))
+)
+	(global_label "VLOGIC_SENSE"
+		(shape passive)
+		(at 124.46 100.33 180)
+		(effects
+			(font
+				(size 1.05 1.05))
+			(justify left))
+)
+	(no_connect
+		(at 119.38 102.87)
+)
+	(no_connect
+		(at 63.5 118.11)
+)
+	(no_connect
+		(at 63.5 120.65)
+)
+	(wire
+		(pts
+			(xy 119.38 133.35)
+			(xy 124.46 133.35))
+		(stroke
+			(width 0)
+			(type default))
+)
+	(global_label "RADIO_RX_MCU"
+		(shape passive)
+		(at 124.46 133.35 180)
+		(effects
+			(font
+				(size 1.05 1.05))
+			(justify left))
+)
+	(wire
+		(pts
+			(xy 119.38 135.89)
+			(xy 124.46 135.89))
+		(stroke
+			(width 0)
+			(type default))
+)
+	(global_label "RADIO_TX_MCU"
+		(shape passive)
+		(at 124.46 135.89 180)
+		(effects
+			(font
+				(size 1.05 1.05))
+			(justify left))
+)
+	(no_connect
+		(at 119.38 138.43)
+)
+	(no_connect
+		(at 119.38 140.97)
+)
+	(wire
+		(pts
+			(xy 119.38 148.59)
+			(xy 124.46 148.59))
+		(stroke
+			(width 0)
+			(type default))
+)
+	(global_label "GPS_FAULT_N"
+		(shape passive)
+		(at 124.46 148.59 180)
+		(effects
+			(font
+				(size 1.05 1.05))
+			(justify left))
+)
+	(text "R10: USART6 PC6/PC7 AF7 GPS; UART5 PB13/PB12 AF14 radio. Port EN and OE default low. EXTI10 GPS_FAULT_N; EXTI9 RADIO_FAULT_N; EXTI12 CAM_FAULT_N; EXTI4 LOGIC_SOURCE_ST (PA4), EXTI5 BAT_FAULT_N (PA5); VLOGIC_SENSE ADC on PA6 (D-R2-09). PE1 remains polled."
+		(at 20.32 259.08 0)
+		(effects
+			(font
