File: m3_design/assembly_review/mcu.kicad_sch (KiCad schematic)
At the start: 21 parts, among them J2 TC2030-IDC-NL SWD, U1 STM32H743VIT6, Y1 25MHz CL8pF

Commit message: R10 single screw-switch arming pass before review round 9
Preparatory single-switch pass, not a full review round or clean-round credit.
Remove J124 and its fused ARM link, join the post-switch bus as RAW_ACT, and
implement the independent PC1 load-switch enable through R122/Q122 while PE4
controls the fire FET. Move R134 for direct bottom-side fire routing. Update
schematic/PCB generators, contracts, seeded tests, binding and operating records.
No interrupted changes were discarded. AUD/GAP cuts and fresh round 9 follow.

Board SHA-256: 60be35eaff86dd7a5fb8e065aa4204a51e7d786d7dfc8d2456cdd66c4b86f901
Board: 46 x 90 mm, 4 layers, 2521622 bytes. Two full builds are byte-identical.
Netlist SHA-256: 3e08722d7ac997131cb11d7c9cb2d25e1b3babcfb853b71230db01118bc70e69
Fab: 228 CPL rows, 83 BOM lines; orientation, paste and manifest checks pass.
Hot-plug: same input-feed signature; 2304 corners and local sensitivities pass
(simulation / Inference). Bench, firmware, RF immunity and physical fit unverified.

Final unskipped tools/check.sh: exit 0
DRC violations 0  unconnected 0  schematic parity 0  ERC 0
metadata / 3D model audit: OK
fit check: OK (CAD envelopes only)
R10 CAD contract (full): OK
routing hygiene: 0 failing, 0 allowlisted, 0 leftovers recorded
actuator safety contract: OK
Fab manifest: OK; 5 outputs match the current CAD and export inputs
Self-tests: shell 4, fit 23, paste 5, route 57; R10 122 (3 NumPy tests
skipped in KiCad Python then passed separately). Standalone plate 3 passed.
Added local absolute paths: 0. No direct Git index/commit mutation performed.

Co-Authored-By: Claude Opus 5.5 <noreply@anthropic.com>
Connections:
- net ACT_EN_MCU: now reaches U1.16 (PC1)
- no-connect marks 30 -> 29
Other:
- note added: "Single screw switch: PC1 U1.16 ACT_EN_MCU drives R122 1k and Q122; initialise low before output mode. R123 100k holds the load switch off at reset. Disable synchronous trace (PC1 TRACED0, PE4 TRACED1); lock and read back both gate GPIO configurations."
Changed lines of the file:
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@@
-)
-	(no_connect
-		(at 119.38 82.55)
 )
 	(no_connect
@@
 			(justify left))
 )
+	(wire
+		(pts
+			(xy 119.38 82.55)
+			(xy 124.46 82.55))
+		(stroke
+			(width 0)
+			(type default))
+)
+	(global_label "ACT_EN_MCU"
+		(shape passive)
+		(at 124.46 82.55 180)
+		(effects
+			(font
+				(size 1.05 1.05))
+			(justify left))
+)
 	(text "R10: USART6 PC6/PC7 AF7 GPS; UART5 PB13/PB12 AF14 radio. Port EN and OE default low. EXTI10 GPS_FAULT_N; EXTI9 RADIO_FAULT_N; EXTI12 CAM_FAULT_N; EXTI4 LOGIC_SOURCE_ST (PA4), EXTI5 BAT_FAULT_N (PA5); VLOGIC_SENSE ADC on PA6 (D-R2-09). EXTI1 PE1 IMU_INT1 data-ready (R6-MCU-01)."
 		(at 20.32 259.08 0)
 		(effects
 			(font
+				(size 1.05 1.05))
+			(justify left))
+)
+	(text "Single screw switch: PC1 U1.16 ACT_EN_MCU drives R122 1k and Q122; initialise low before output mode. R123 100k holds the load switch off at reset. Disable synchronous trace (PC1 TRACED0, PE4 TRACED1); lock and read back both gate GPIO configurations."
+		(at 20.32 269.24 0)
+		(effects
+			(font

Commit message: R10 requirements-audit cuts and GAP fixes before review round 9
Implement adopted AUD-1 through AUD-10 and GAP-1 through GAP-5 after the single-switch pass.
Remove the advisory pull-pin, redundant probes and GPS/radio IO LDO cells; qualify the smaller
AONR21357 pair, correct C120 voltage rating, standardize shared-code capacitor lands, simplify
slow returns and fire-only copper, localize U9 output protection and add exactly two U401 VIPPO vias.
Record physical-current timing, coupled fire/source budget, C84 manual fitting and narrowed gate scopes.

Board SHA-256: 877d01996a59e9dd5c6dbc367274bb9a323a13982d67960fe46df9b0ee53205d
Board: 46 x 90 mm, 4 layers, 2365477 bytes; 225 footprints, 883 straight tracks, 323 vias.
Netlist SHA-256: 0843da709e2d7a757e9b35cdff48158a54012c5353619cbf409ab961efd2c3ca
Two fresh complete passing builds are byte-identical. Schematic: 700 pins; 22 seeded faults detected.

Final unskipped tools/check.sh: exit 0
DRC violations 0  unconnected 0  schematic parity 0  ERC 0
metadata / 3D model audit: OK
silkscreen outside the board outline: 0 stroke points
fit check: OK (CAD envelopes only)
R10 CAD contract (full): OK
routing hygiene: 0 failing, 0 allowlisted, 0 leftovers recorded
actuator safety contract: OK
Fab manifest: OK; 5 outputs match current CAD and export inputs
Self-tests: shell 4, fit 24, paste 5, routing 59, R10 131; three NumPy cases rerun and passed.

Fab: 215 CPL rows, 82 BOM codes; orientation / paste / manifest pass. Hot-plug: 2304 required
cases plus convergence and controls pass (simulation / Inference). Plate f1 280.9 Hz (Inference).
Live JLC: $84.43 vs $84.41 target, 46 Extended codes; R430 / U4 short. Procurement exit 1 is a
disclosed OQ-3 / ordering deviation, not a CAD gate pass. No quote accepted or order placed.
Firmware, bench, thermal/transient correlation, process acceptance, installed RF immunity and physical fit unverified.

This preparatory pass earns no clean-review credit. Start fresh full ten-lens round 9 on th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
Connections:
- net PULLPIN: no longer names the net of U1.7 (PC13)
- no-connect marks 29 -> 30
Other:
- note added: "Single screw switch: PC1 U1.16 ACT_EN_MCU drives R122 1k and Q122; initialise low before output mode. R123 100k holds the load switch off at reset. Hold PE4 low for >=100 ms after ACT_EN before bus checks. Disable synchronous trace (PC1 TRACED0, PE4 TRACED1); lock/read back both gate GPIO configurations. AUD-4: PC13 U1.7 is NC/analog; no pull-pin."
- note removed: "Single screw switch: PC1 U1.16 ACT_EN_MCU drives R122 1k and Q122; initialise low before output mode. R123 100k holds the load switch off at reset. Disable synchronous trace (PC1 TRACED0, PE4 TRACED1); lock and read back both gate GPIO configurations."
Changed lines of the file:
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@@
 	(wire
 		(pts
-			(xy 63.5 77.47)
-			(xy 58.42 77.47))
-		(stroke
-			(width 0)
-			(type default))
-)
-	(global_label "PULLPIN"
-		(shape passive)
-		(at 58.42 77.47 0)
-		(effects
-			(font
-				(size 1.05 1.05))
-			(justify right))
-)
-	(wire
-		(pts
 			(xy 63.5 80.01)
 			(xy 58.42 80.01))
@@
 )
 	(no_connect
+		(at 63.5 77.47)
+)
+	(no_connect
 		(at 63.5 92.71)
 )
@@
 			(justify left))
 )
-	(text "Single screw switch: PC1 U1.16 ACT_EN_MCU drives R122 1k and Q122; initialise low before output mode. R123 100k holds the load switch off at reset. Disable synchronous trace (PC1 TRACED0, PE4 TRACED1); lock and read back both gate GPIO configurations."
+	(text "Single screw switch: PC1 U1.16 ACT_EN_MCU drives R122 1k and Q122; initialise low before output mode. R123 100k holds the load switch off at reset. Hold PE4 low for >=100 ms after ACT_EN before bus checks. Disable synchronous trace (PC1 TRACED0, PE4 TRACED1); lock/read back both gate GPIO configurations. AUD-4: PC13 U1.7 is NC/analog; no pull-pin."
 		(at 20.32 269.24 0)
 		(effects

Commit message: Finish R10 round 9 Minor fix pass
Complete the interrupted generator rebuild and apply the recorded round 9
Minor fixes: capacitor labels, cold-screen ordering, debugger instructions,
local route cleanups, gate fault detection and explicit R10 procurement limits.
Refresh the board-bound fabrication, supplier and validation records.

Round 9 reviewed 8bccb07: 0 Critical, 0 Major, 21 Minor groups. Round 10 will
freshly review this committed fix pass, including every changed CAD item.

Board SHA-256: b337fe63c258c85ba4120e75ad018afa0c22241f8bc21a4172787cf2887208d9
Board: 46 x 90 mm, 2366509 bytes. Two COMPLETE builds pass; all 21 generated
CAD and binding files are byte-identical.

Unskipped tools/check.sh: exit 0.
DRC violations 0; unconnected 0; schematic parity 0; ERC 0.
Metadata / 3D, silk, fit / plate, all 33 R10 rules, routing hygiene, actuator
contract and current 5-output fabrication manifest: OK.
Self-tests: shell 4, procurement 19, fit 24, paste 5, routing 59, R10 140;
3 NumPy cases rerun successfully, no unresolved skips. Hot-plug: 2304/2304
required cases pass (simulation / Inference).

Fab export, required fitting, orientation and paste pass: 215 CPL rows,
82 BOM codes. Fresh supplier/procurement checks correctly FAIL the known
$84.43 versus $84.41 cap and R430/U4 stock shortages; 46 Extended codes.
OQ-3 and final deviation acceptance remain pending. No firmware, bench,
installed RF immunity, physical fit, assembly-process or flight result claimed.

Evidence: docs/R10_VALIDATION.md and sources/r10_review/round9_fix_validation.json
and round9_fix_check.txt under m3_design/assembly_review. Native headless
KiCad environment uses the external D-R1-05 mouse-query workaround only;
repository gates and CAD rules are unchanged by that workaround.

Co-Authored-By: Claude Opus 5.5 <noreply@anthropic.com>
Parts:
- C19, C20: value 2.2uF -> 2.2uF 16V X5R 10%
- C22: value 1uF -> 1uF 50V X5R 10%
- C23: value 4.7uF -> 4.7uF 16V X5R 10%
- C25, C26: value 10pF -> 10pF 50V C0G 5%
Other:
- note added: "Single screw switch: PC1 U1.16 ACT_EN_MCU drives R122 1k and Q122; initialise PC1 and PE4 low before output mode. R123 100k holds the load switch off at reset. Both low for passive cold screening; after prior enable wait >=1 s and verify bus discharge. Refuse ground faults BEFORE PC1 enable; then PC1 high, PE4 low >=100 ms before powered-bus checks (D-SS-04). Disable synchronous trace; lock/read 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"
- note removed: "Single screw switch: PC1 U1.16 ACT_EN_MCU drives R122 1k and Q122; initialise low before output mode. R123 100k holds the load switch off at reset. Hold PE4 low for >=100 ms after ACT_EN before bus checks. Disable synchronous trace (PC1 TRACED0, PE4 TRACED1); lock/read back both gate GPIO configurations. AUD-4: PC13 U1.7 is NC/analog; no pull-pin."
Changed lines of the file:
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@@
 					(size 1.27 1.27))
 				(justify left)))
-		(property "Value" "2.2uF"
+		(property "Value" "2.2uF 16V X5R 10%"
 			(at 210.82 181.60999999999999 0)
 			(effects
@@
 					(size 1.27 1.27))
 				(justify left)))
-		(property "Value" "2.2uF"
+		(property "Value" "2.2uF 16V X5R 10%"
 			(at 256.54 181.60999999999999 0)
 			(effects
@@
 					(size 1.27 1.27))
 				(justify left)))
-		(property "Value" "1uF"
+		(property "Value" "1uF 50V X5R 10%"
 			(at 332.74 181.60999999999999 0)
 			(effects
@@
 					(size 1.27 1.27))
 				(justify left)))
-		(property "Value" "4.7uF"
+		(property "Value" "4.7uF 16V X5R 10%"
 			(at 363.22 181.60999999999999 0)
 			(effects
@@
 					(size 1.27 1.27))
 				(justify left)))
-		(property "Value" "10pF"
+		(property "Value" "10pF 50V C0G 5%"
 			(at 220.98 105.41000000000001 0)
 			(effects
@@
 					(size 1.27 1.27))
 				(justify left)))
-		(property "Value" "10pF"
+		(property "Value" "10pF 50V C0G 5%"
 			(at 251.45999999999998 105.41000000000001 0)
 			(effects
@@
 			(justify left))
 )
-	(text "Single screw switch: PC1 U1.16 ACT_EN_MCU drives R122 1k and Q122; initialise low before output mode. R123 100k holds the load switch off at reset. Hold PE4 low for >=100 ms after ACT_EN before bus checks. Disable synchronous trace (PC1 TRACED0, PE4 TRACED1); lock/read back both gate GPIO configurations. AUD-4: PC13 U1.7 is NC/analog; no pull-pin."
+	(text "Single screw switch: PC1 U1.16 ACT_EN_MCU drives R122 1k and Q122; initialise PC1 and PE4 low before output mode. R123 100k holds the load switch off at reset. Both low for passive cold screening; after prior enable wait >=1 s and verify bus discharge. Refuse ground faults BEFORE PC1 enable; then PC1 high, PE4 low >=100 ms before powered-bus checks (D-SS-04). Disable synchronous trace; lock/read back both gate GPIO configurations. AUD-4: PC13 U1.7 is NC/analog; no pull-pin."
 		(at 20.32 269.24 0)
 		(effects
