File: m3_design/assembly_review/camera_connector.kicad_sch (KiCad schematic)
At the start: 5 parts, among them J9 CAM 5V / GND / RX / TX

Commit message: Validate and harden R5 flight computer CAD
Parts:
- J9: Manufacturer (none) -> DORABO; Manufacturer Part (none) -> DB128V-5.08-4P-GN-S
Changed lines of the file:
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@@
+				(font
+					(size 1.27 1.27))))
+		(property "Manufacturer" "DORABO"
+			(at 76.2 88.9 0)
+			(hide yes)
+			(effects
+				(font
+					(size 1.27 1.27))))
+		(property "Manufacturer Part" "DB128V-5.08-4P-GN-S"
+			(at 76.2 88.9 0)
+			(hide yes)
+			(effects
 				(font
 					(size 1.27 1.27))))

Commit message: Complete R6 flight computer CAD and validated fabrication package
Add protected radio and GPS ports, reset-off port power, compact connectors and single-channel pyro layout. Close independent routing, ground-return and decoupling findings; record zero-error CAD checks and current manufacturing artifacts. Document 100 mm length, IMU stock hold and remaining firmware and hardware qualification.
Parts:
- J9: value CAM 5V / GND / RX / TX -> CAMERA 5V/GND/RX/TX; footprint rocket:M3_DB128V_4P -> rocket:M3_GH_BM04B_GHS_TBT; LCSC C2915641 -> C161692; LCSC Part (none) -> C161692; Manufacturer DORABO -> JST; Manufacturer Part DB128V-5.08-4P-GN-S -> BM04B-GHS-TBT(LF)(SN)
Changed lines of the file:
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@@
 		(title "06 | Camera terminal and characterization")
 		(date "2026-09-07")
-		(rev "M3-ASSY-R4")
+		(rev "M3-ASSY-R6")
 		(company "Single-board M3 candidate; full system incomplete"))
 	(text "06 | Camera terminal and characterization"
@@
 				(font
 					(size 1.27 1.27))))
-		(property "Value" "CAM 5V / GND / RX / TX"
+		(property "Value" "CAMERA 5V/GND/RX/TX"
 			(at 76.2 81.28 0)
 			(effects
 				(font
 					(size 1.27 1.27))))
-		(property "Footprint" "rocket:M3_DB128V_4P"
+		(property "Footprint" "rocket:M3_GH_BM04B_GHS_TBT"
 			(at 76.2 88.9 0)
 			(hide yes)
@@
 				(font
 					(size 1.27 1.27))))
-		(property "LCSC" "C2915641"
+		(property "LCSC" "C161692"
 			(at 76.2 88.9 0)
 			(hide yes)
@@
 				(font
 					(size 1.27 1.27))))
-		(property "Manufacturer" "DORABO"
+		(property "Manufacturer" "JST"
 			(at 76.2 88.9 0)
 			(hide yes)
@@
 				(font
 					(size 1.27 1.27))))
-		(property "Manufacturer Part" "DB128V-5.08-4P-GN-S"
+		(property "Manufacturer Part" "BM04B-GHS-TBT(LF)(SN)"
 			(at 76.2 88.9 0)
 			(hide yes)
@@
 				(path "/6007a7db-6a58-5660-8beb-956dea045ff8/df8afa2f-b72f-56f6-9fee-55c91cce0fe4"
 					(reference "J9")
-					(unit 1)))))
+					(unit 1))))		(property "LCSC Part" "C161692"
+			(at 0 0 0)
+			(hide yes)
+			(effects
+				(font
+					(size 1.27 1.27))
+				(justify left)))
+)
 	(wire
 		(pts
