File: m3_design/assembly_review/camera_connector.kicad_sch (KiCad schematic)
At the start: 5 parts, among them J9 CAMERA 5V/GND/RX/TX

Commit message: R10: m3_design/r10_build.sh and per-family stage gate; m3_design/assembly_review rebuilt as M3-ASSY-R10 (board 883d2db5..., 46 x 90 mm); tools/check.sh passes at zero; binding note bound to the board
Co-Authored-By: Claude Opus 5.5 <noreply@anthropic.com>
Parts:
- removed TP72: CAM_5V, rocket:M3_TestPad_1.5, symbol M3:TestPoint
- removed TP75: CAM_RX_TEST, rocket:M3_TestPad_1.5, symbol M3:TestPoint
- removed TP76: CAM_TX_TEST, rocket:M3_TestPad_1.5, symbol M3:TestPoint
Other:
- note added: "R10 camera GH port: regulated switched supply, GND, camera RX and camera TX. UART isolation remains on sheet09."
- note added: "The5 redundant camera characterization pads were removed; probe the connector or fitted circuitry. No pyro/arming test pads changed."
- note removed: "06 | Camera terminal and characterization"
- note removed: "3.3V signalling candidate. Actual camera thresholds and power-off leakage need measurement."
- note removed: "Battery entry added in PWR-R1; dynamic/thermal/USB qualification is pending."
- note removed: "Camera power toggling can corrupt recording: stop recording before normal shutdown."
- note removed: "J9 is a dedicated camera output, not a generic USB 5 V source."
- note removed: "Measure TP73 with >=10 Mohm input; loading ILM alters the current limit."
- note removed: "Pin 1: regulated power. Pin 2: GND. Pin 3: from camera TX. Pin 4: to camera RX."
- note removed: "Pins 3/4: UART through U12; TP75/76 remain wire-side measurement points."
- note removed: "RunCam manual: 5-20 V regulated input; source capability >=1 A; max 450 mA at 5 V."
- note removed: "TP70 -> TP71 -> TP72 localizes input / eFuse / regulator faults."
- note removed: "This is an engineering candidate; it is not released for fabrication or flight."
Changed lines of the file:
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@@
 		(title "06 | Camera terminal and characterization")
 		(date "2026-09-07")
-		(rev "M3-ASSY-R9")
+		(rev "M3-ASSY-R10")
 		(company "Single-board M3 candidate; full system incomplete"))
-	(text "06 | Camera terminal and characterization"
-		(at 20.32 20.32 0)
-		(effects
-			(font
-				(size 2.54 2.54))
-			(justify left))
-)
 	(symbol
 		(lib_id "M3:CameraTerminal")
@@
 	(symbol
 		(lib_id "M3:TestPoint")
-		(at 170.18 58.42 0)
-		(unit 1)
-		(in_bom no)
-		(on_board yes)
-		(dnp no)
-		(property "Reference" "TP72"
-			(at 170.18 50.800000000000004 0)
-			(effects
-				(font
-					(size 1.27 1.27))))
-		(property "Value" "CAM_5V"
-			(at 170.18 54.61000000000001 0)
-			(effects
-				(font
-					(size 1.27 1.27))))
-		(property "Footprint" "rocket:M3_TestPad_1.5"
-			(at 170.18 58.42 0)
-			(hide yes)
-			(effects
-				(font
-					(size 1.27 1.27))))
-		(property "Datasheet" ""
-			(at 170.18 58.42 0)
-			(hide yes)
-			(effects
-				(font
-					(size 1.27 1.27))))
-		(property "LCSC" ""
-			(at 170.18 58.42 0)
-			(hide yes)
-			(effects
-				(font
-					(size 1.27 1.27))))
-		(instances
-			(project "m3"
-				(path "/6007a7db-6a58-5660-8beb-956dea045ff8/df8afa2f-b72f-56f6-9fee-55c91cce0fe4"
-					(reference "TP72")
-					(unit 1)))))
-	(wire
-		(pts
-			(xy 170.18 58.42)
-			(xy 162.56 58.42))
-		(stroke
-			(width 0)
-			(type default))
-)
-	(global_label "CAM_5V"
-		(shape passive)
-		(at 162.56 58.42 0)
-		(effects
-			(font
-				(size 1.05 1.05))
-			(justify right))
-)
-	(symbol
-		(lib_id "M3:TestPoint")
 		(at 170.18 88.9 0)
 		(unit 1)
@@
 			(justify right))
 )
-	(symbol
-		(lib_id "M3:TestPoint")
-		(at 170.18 119.38 0)
-		(unit 1)
-		(in_bom no)
-		(on_board yes)
-		(dnp no)
-		(property "Reference" "TP75"
-			(at 170.18 111.75999999999999 0)
-			(effects
-				(font
-					(size 1.27 1.27))))
-		(property "Value" "CAM_RX_TEST"
-			(at 170.18 115.57 0)
-			(effects
-				(font
-					(size 1.27 1.27))))
-		(property "Footprint" "rocket:M3_TestPad_1.5"
-			(at 170.18 119.38 0)
-			(hide yes)
-			(effects
-				(font
-					(size 1.27 1.27))))
-		(property "Datasheet" ""
-			(at 170.18 119.38 0)
-			(hide yes)
-			(effects
-				(font
-					(size 1.27 1.27))))
-		(property "LCSC" ""
-			(at 170.18 119.38 0)
-			(hide yes)
-			(effects
-				(font
-					(size 1.27 1.27))))
-		(instances
-			(project "m3"
-				(path "/6007a7db-6a58-5660-8beb-956dea045ff8/df8afa2f-b72f-56f6-9fee-55c91cce0fe4"
-					(reference "TP75")
-					(unit 1)))))
-	(wire
-		(pts
-			(xy 170.18 119.38)
-			(xy 162.56 119.38))
-		(stroke
-			(width 0)
-			(type default))
-)
-	(global_label "CAM_RX_WIRE"
-		(shape passive)
-		(at 162.56 119.38 0)
+	(text "R10 camera GH port: regulated switched supply, GND, camera RX and camera TX. UART isolation remains on sheet09."
+		(at 20.32 15.24 0)
 		(effects
 			(font
 				(size 1.05 1.05))
-			(justify right))
+			(justify left))
 )
-	(symbol
-		(lib_id "M3:TestPoint")
-		(at 170.18 149.86 0)
-		(unit 1)
-		(in_bom no)
-		(on_board yes)
-		(dnp no)
-		(property "Reference" "TP76"
-			(at 170.18 142.24 0)
-			(effects
-				(font
-					(size 1.27 1.27))))
-		(property "Value" "CAM_TX_TEST"
-			(at 170.18 146.05 0)
-			(effects
-				(font
-					(size 1.27 1.27))))
-		(property "Footprint" "rocket:M3_TestPad_1.5"
-			(at 170.18 149.86 0)
-			(hide yes)
-			(effects
-				(font
-					(size 1.27 1.27))))
-		(property "Datasheet" ""
-			(at 170.18 149.86 0)
-			(hide yes)
-			(effects
-				(font
-					(size 1.27 1.27))))
-		(property "LCSC" ""
-			(at 170.18 149.86 0)
-			(hide yes)
-			(effects
-				(font
-					(size 1.27 1.27))))
-		(instances
-			(project "m3"
-				(path "/6007a7db-6a58-5660-8beb-956dea045ff8/df8afa2f-b72f-56f6-9fee-55c91cce0fe4"
-					(reference "TP76")
-					(unit 1)))))
-	(wire
-		(pts
-			(xy 170.18 149.86)
-			(xy 162.56 149.86))
-		(stroke
-			(width 0)
-			(type default))
-)
-	(global_label "CAM_TX_WIRE"
-		(shape passive)
-		(at 162.56 149.86 0)
+	(text "The5 redundant camera characterization pads were removed; probe the connector or fitted circuitry. No pyro/arming test pads changed."
+		(at 20.32 20.32 0)
 		(effects
 			(font
 				(size 1.05 1.05))
-			(justify right))
-)
-	(text "J9 is a dedicated camera output, not a generic USB 5 V source."
-		(at 20.32 180.34 0)
-		(effects
-			(font
-				(size 1.27 1.27))
 			(justify left))
 )
-	(text "Pin 1: regulated power. Pin 2: GND. Pin 3: from camera TX. Pin 4: to camera RX."
-		(at 20.32 187.96 0)
-		(effects
-			(font
-				(size 1.27 1.27))
-			(justify left))
-)
-	(text "Pins 3/4: UART through U12; TP75/76 remain wire-side measurement points."
-		(at 20.32 195.58 0)
-		(effects
-			(font
-				(size 1.27 1.27))
-			(justify left))
-)
-	(text "3.3V signalling candidate. Actual camera thresholds and power-off leakage need measurement."
-		(at 20.32 203.2 0)
-		(effects
-			(font
-				(size 1.27 1.27))
-			(justify left))
-)
-	(text "Battery entry added in PWR-R1; dynamic/thermal/USB qualification is pending."
-		(at 20.32 210.82 0)
-		(effects
-			(font
-				(size 1.27 1.27))
-			(justify left))
-)
-	(text "TP70 -> TP71 -> TP72 localizes input / eFuse / regulator faults."
-		(at 20.32 218.44 0)
-		(effects
-			(font
-				(size 1.27 1.27))
-			(justify left))
-)
-	(text "Measure TP73 with >=10 Mohm input; loading ILM alters the current limit."
-		(at 20.32 226.06 0)
-		(effects
-			(font
-				(size 1.27 1.27))
-			(justify left))
-)
-	(text "Camera power toggling can corrupt recording: stop recording before normal shutdown."
-		(at 20.32 233.68 0)
-		(effects
-			(font
-				(size 1.27 1.27))
-			(justify left))
-)
-	(text "RunCam manual: 5-20 V regulated input; source capability >=1 A; max 450 mA at 5 V."
-		(at 20.32 241.3 0)
-		(effects
-			(font
-				(size 1.27 1.27))
-			(justify left))
-)
-	(text "This is an engineering candidate; it is not released for fabrication or flight."
-		(at 20.32 248.92000000000002 0)
-		(effects
-			(font
-				(size 1.27 1.27))
-			(justify left))
-)
