File: m3_design/assembly_review/camera_power.kicad_sch (KiCad schematic)
At the start: 22 parts, among them U7 TPS259570DSGR, U8 AP63301WU-7

Commit message: Validate and harden R5 flight computer CAD
Parts:
- U7: Manufacturer (none) -> Texas Instruments; Manufacturer Part (none) -> TPS259570DSGR
Changed lines of the file:
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@@
+				(font
+					(size 1.27 1.27))))
+		(property "Manufacturer" "Texas Instruments"
+			(at 83.82 76.2 0)
+			(hide yes)
+			(effects
+				(font
+					(size 1.27 1.27))))
+		(property "Manufacturer Part" "TPS259570DSGR"
+			(at 83.82 76.2 0)
+			(hide yes)
+			(effects
 				(font
 					(size 1.27 1.27))))
