File: m3_design/assembly_review/pullpin_buzzer.kicad_sch (KiCad schematic)
At the start: 10 parts, among them J123 PULL-PIN PH 1x2, Q123 AO3400A

Commit message: Validate and harden R5 flight computer CAD
Parts:
- C160: Manufacturer (none) -> Samsung Electro-Mechanics; Manufacturer Part (none) -> CL05B104KO5NNNC
- R160: Manufacturer (none) -> UNI-ROYAL(Uniroyal Elec); Manufacturer Part (none) -> 0402WGF1001TCE
- R161, R163: Manufacturer (none) -> UNI-ROYAL(Uniroyal Elec); Manufacturer Part (none) -> 0402WGF1002TCE
- R162: Manufacturer (none) -> UNI-ROYAL(Uniroyal Elec); Manufacturer Part (none) -> 0805W8F2200T5E
Changed lines of the file:
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@@
+				(font
+					(size 1.27 1.27))))
+		(property "Manufacturer" "UNI-ROYAL(Uniroyal Elec)"
+			(at 99.06 50.8 0)
+			(hide yes)
+			(effects
+				(font
+					(size 1.27 1.27))))
+		(property "Manufacturer Part" "0402WGF1001TCE"
+			(at 99.06 50.8 0)
+			(hide yes)
+			(effects
 				(font
 					(size 1.27 1.27))))
@@
 				(font
 					(size 1.27 1.27))))
+		(property "Manufacturer" "UNI-ROYAL(Uniroyal Elec)"
+			(at 157.48 50.8 0)
+			(hide yes)
+			(effects
+				(font
+					(size 1.27 1.27))))
+		(property "Manufacturer Part" "0402WGF1002TCE"
+			(at 157.48 50.8 0)
+			(hide yes)
+			(effects
+				(font
+					(size 1.27 1.27))))
 		(instances
 			(project "m3"
@@
 				(font
 					(size 1.27 1.27))))
+		(property "Manufacturer" "Samsung Electro-Mechanics"
+			(at 215.9 50.8 0)
+			(hide yes)
+			(effects
+				(font
+					(size 1.27 1.27))))
+		(property "Manufacturer Part" "CL05B104KO5NNNC"
+			(at 215.9 50.8 0)
+			(hide yes)
+			(effects
+				(font
+					(size 1.27 1.27))))
 		(instances
 			(project "m3"
@@
 				(font
 					(size 1.27 1.27))))
+		(property "Manufacturer" "UNI-ROYAL(Uniroyal Elec)"
+			(at 157.48 114.3 0)
+			(hide yes)
+			(effects
+				(font
+					(size 1.27 1.27))))
+		(property "Manufacturer Part" "0805W8F2200T5E"
+			(at 157.48 114.3 0)
+			(hide yes)
+			(effects
+				(font
+					(size 1.27 1.27))))
 		(instances
 			(project "m3"
@@
 			(at 215.9 114.3 0)
 			(hide yes)
+			(effects
+				(font
+					(size 1.27 1.27))))
+		(property "Manufacturer" "UNI-ROYAL(Uniroyal Elec)"
+			(at 215.9 114.3 0)
+			(hide yes)
+			(effects
+				(font
+					(size 1.27 1.27))))
+		(property "Manufacturer Part" "0402WGF1002TCE"
+			(at 215.9 114.3 0)
+			(hide yes)

Commit message: Complete R6 flight computer CAD and validated fabrication package
Add protected radio and GPS ports, reset-off port power, compact connectors and single-channel pyro layout. Close independent routing, ground-return and decoupling findings; record zero-error CAD checks and current manufacturing artifacts. Document 100 mm length, IMU stock hold and remaining firmware and hardware qualification.
Parts:
- C160: value 100nF -> 100nF 50V X7R 10%; LCSC C1525 -> C307331; LCSC Part (none) -> C307331; Manufacturer Part CL05B104KO5NNNC -> CL05B104KB54PNC
- LS120: value MLT-8530 -> MLT-5020; footprint rocket:BUZ-SMD_4P-L8.5-W8.5-P8.50-BR -> rocket:M3_MLT5020_3pad; symbol M3:Buzzer_4pad -> M3:Buzzer_3pad; LCSC C94599 -> C94598; LCSC Part (none) -> C94598; Manufacturer Part MLT-8530 -> MLT-5020
Connections:
- no-connect marks 2 -> 1
Other:
- note added: "BUZZ_DRV = PA5 (pin 29). MLT-5020: 4 kHz, 50% duty; software toggle or TIM8_CH1N (AF3). Never leave the coil driven with DC."
- note added: "LS120 MLT-5020: pad 1 = +, pad 2 = -, pad 3 = isolated mechanical tab. Huaneng 2021-05-27 drawing; body 5.0 +/-0.3 mm, height 2.0 +/-0.2 mm."
- note removed: "BUZZ_DRV = PA5 (pin 29), moved off PE6 (P1-10). 2.7 kHz 50 % duty, software toggle or TIM8_CH1N (AF3, verified, M3_R3 6). Never TIM2."
- note removed: "LS120 MLT-8530: pad 1 = + lead, pad 2 = - lead, pads 3/4 = dummy (Huaneng spec 5.2). Closes CIRCUIT_REVIEW 3.4."
Changed lines of the file:
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@@
 		(title "14 | Launch pull-pin and buzzer")
 		(date "2026-09-25")
-		(rev "M3-ASSY-R4")
+		(rev "M3-ASSY-R6")
 		(company "Single-board M3 candidate; actuator merge, not bench-verified"))
 	(symbol
@@
 					(size 1.27 1.27))
 				(justify left)))
-		(property "Value" "100nF"
+		(property "Value" "100nF 50V X7R 10%"
 			(at 219.71 59.69 0)
 			(effects
@@
 				(font
 					(size 1.27 1.27))))
-		(property "LCSC" "C1525"
+		(property "LCSC" "C307331"
 			(at 215.9 50.8 0)
 			(hide yes)
@@
 				(font
 					(size 1.27 1.27))))
-		(property "Manufacturer Part" "CL05B104KO5NNNC"
+		(property "Manufacturer Part" "CL05B104KB54PNC"
 			(at 215.9 50.8 0)
 			(hide yes)
@@
 				(path "/6007a7db-6a58-5660-8beb-956dea045ff8/5ee931eb-d962-5c64-b0fd-46233c13323f"
 					(reference "C160")
-					(unit 1)))))
+					(unit 1))))		(property "LCSC Part" "C307331"
+			(at 0 0 0)
+			(hide yes)
+			(effects
+				(font
+					(size 1.27 1.27))
+				(justify left)))
+)
 	(wire
 		(pts
@@
 )
 	(symbol
-		(lib_id "M3:Buzzer_4pad")
+		(lib_id "M3:Buzzer_3pad")
 		(at 332.74 50.8 0)
 		(unit 1)
@@
 					(size 1.27 1.27))
 				(justify left)))
-		(property "Value" "MLT-8530"
+		(property "Value" "MLT-5020"
 			(at 336.55 59.69 0)
 			(effects
@@
 					(size 1.27 1.27))
 				(justify left)))
-		(property "Footprint" "rocket:BUZ-SMD_4P-L8.5-W8.5-P8.50-BR"
+		(property "Footprint" "rocket:M3_MLT5020_3pad"
 			(at 332.74 50.8 0)
 			(hide yes)
@@
 				(font
 					(size 1.27 1.27))))
-		(property "Datasheet" ""
+		(property "Datasheet" "https://datasheet.lcsc.com/datasheet/pdf/23f5c6599ed9cb614c21ac31ad2b1106.pdf"
 			(at 332.74 50.8 0)
 			(hide yes)
@@
 				(font
 					(size 1.27 1.27))))
-		(property "LCSC" "C94599"
+		(property "LCSC" "C94598"
 			(at 332.74 50.8 0)
 			(hide yes)
@@
 				(font
 					(size 1.27 1.27))))
-		(property "Manufacturer Part" "MLT-8530"
+		(property "Manufacturer Part" "MLT-5020"
 			(at 332.74 50.8 0)
 			(hide yes)
@@
 				(path "/6007a7db-6a58-5660-8beb-956dea045ff8/5ee931eb-d962-5c64-b0fd-46233c13323f"
 					(reference "LS120")
-					(unit 1)))))
+					(unit 1))))		(property "LCSC Part" "C94598"
+			(at 0 0 0)
+			(hide yes)
+			(effects
+				(font
+					(size 1.27 1.27))
+				(justify left)))
+)
 	(wire
 		(pts
@@
 	(no_connect
 		(at 342.9 48.26)
-)
-	(no_connect
-		(at 342.9 53.34)
 )
 	(symbol
@@
 			(justify left))
 )
-	(text "LS120 MLT-8530: pad 1 = + lead, pad 2 = - lead, pads 3/4 = dummy (Huaneng spec 5.2). Closes CIRCUIT_REVIEW 3.4."
+	(text "LS120 MLT-5020: pad 1 = +, pad 2 = -, pad 3 = isolated mechanical tab. Huaneng 2021-05-27 drawing; body 5.0 +/-0.3 mm, height 2.0 +/-0.2 mm."
 		(at 20.32 260.24 0)
 		(effects
@@
 			(justify left))
 )
-	(text "BUZZ_DRV = PA5 (pin 29), moved off PE6 (P1-10). 2.7 kHz 50 % duty, software toggle or TIM8_CH1N (AF3, verified, M3_R3 6). Never TIM2."
+	(text "BUZZ_DRV = PA5 (pin 29). MLT-5020: 4 kHz, 50% duty; software toggle or TIM8_CH1N (AF3). Never leave the coil driven with DC."
 		(at 20.32 267.86 0)
 		(effects
