File: m3_design/assembly_review/pyro.kicad_sch (KiCad schematic)
At the start: 43 parts, among them J120 ARM CH2: RAW / BUS2, J121 IGNITER 1: E1- / E1+, J124 ARM CH1: BUS1 / RAW, J125 IGNITER 2: E2+ / E2-, Q124 AON7524, Q125 AON7524

Commit message: Validate and harden R5 flight computer CAD
Parts:
- C127, C129, C139, C141: Manufacturer (none) -> FH (Guangdong Fenghua Advanced Tech); Manufacturer Part (none) -> 0603B103K500NT
- R126, R138: Manufacturer (none) -> UNI-ROYAL(Uniroyal Elec); Manufacturer Part (none) -> 0805W8F2200T5E
- R127, R139: Manufacturer (none) -> UNI-ROYAL(Uniroyal Elec); Manufacturer Part (none) -> 0402WGF1001TCE
- R128, R131, R140, R143: Manufacturer (none) -> UNI-ROYAL(Uniroyal Elec); Manufacturer Part (none) -> 0402WGF1002TCE
- R129, R132, R141, R144, R173, R174, R175, R176: Manufacturer (none) -> UNI-ROYAL(Uniroyal Elec); Manufacturer Part (none) -> 0402WGF5101TCE
- R130, R133, R142, R145, R178, R179, R180, R181: Manufacturer (none) -> UNI-ROYAL(Uniroyal Elec); Manufacturer Part (none) -> 0402WGF2001TCE

Commit message: Complete R6 flight computer CAD and validated fabrication package
Add protected radio and GPS ports, reset-off port power, compact connectors and single-channel pyro layout. Close independent routing, ground-return and decoupling findings; record zero-error CAD checks and current manufacturing artifacts. Document 100 mm length, IMU stock hold and remaining firmware and hardware qualification.
Parts:
- removed C138: 220nF 25V X7R, rocket:C0603, symbol M3:C
- removed C139, C141: 10nF, rocket:C0603, symbol M3:C
- removed C140: 100nF 50V X7R 10%, rocket:C_0603_1608Metric, symbol M3:C
- removed J120: ARM CH2: RAW / BUS2, rocket:M3_DB128L_2P_BK, symbol M3:Conn_1x2
- removed J125: IGNITER 2: E2+ / E2-, rocket:M3_DB128L_2P, symbol M3:Conn_1x2
- removed Q125: AON7524, rocket:M3_AON7524_DFN3x3A, symbol M3:NMOS_DFN8EP
- removed R135: 2R 1% 2W pulse, rocket:R2512, symbol M3:R
- removed R138: 220R, rocket:R0805, symbol M3:R
- removed R139: 1k, rocket:R0402, symbol M3:R
- removed R140, R143: 10k, rocket:R0402, symbol M3:R
- removed R141, R144, R174, R176: 5.1k, rocket:R0402, symbol M3:R
- removed R142, R145, R179, R181: 2k, rocket:R0402, symbol M3:R
- removed TP123: PYRO2_GATE, rocket:M3_TestPad_1.5, symbol M3:TestPoint
- J121: footprint rocket:M3_DB128L_2P -> rocket:M3_DB128L_2P_BK; LCSC C430603 -> C430601; LCSC Part C430603 -> C430601; Manufacturer Part DB128L-5.08-2P-OG-S -> DB128L-5.08-2P-BK-S
Connections:
- net PYRO2_COLD: no longer names the net of D120.2 (K2)
- no-connect marks 0 -> 1
Other:
- note added: "12 | Single pyro CH1, arming and continuity"
- note added: "CONT: R173 + R129 over R130 || R178 from drain. ARM: R132 + R175 over R133 || R180 from fused bus."
- note added: "D120 cathode 1 + R131 10k: cold pull-up for plug-out FET-short detection. Cathode 2 NC. In flight: log only, never veto."
- note added: "Igniter across J121.1 OUT and J121.2 IGN. J124 and J121 pin ordering is retained from the reviewed CH1."
- note added: "One pyro channel. J124.2 RAW -> external F1 5A FAST -> J124.1 BUS1. Black J124 ARM / J121 IGN; identify by silk and pin legends."
- note added: "R134: 2 ohm 2 W pulse-rated Bourns CRM2512; shorted-igniter current about 4 A. Firmware fire pulse <= 20 ms."
- note added: "Split divider tops: R173 + R129 and R132 + R175 (2 x 5.1k). Bottoms: R130 || R178 and R133 || R180 (2 x 2k). Ratio 1/11.2. R168/R170 4.7k at MCU. CH1 coating and safety rules A-H/A2 remain mandatory."
- note added: "With the ARM plug out NOTHING connects RAW_ACT to PYRO1_BUS. No test point on BUS, IGN or OUT."
- note removed: "12 | Pyro channels, arming and continuity"
- note removed: "CONT = (2 x 5.1k)/(2 x 2k parallel) from each drain (open detector only, CIRCUIT_REVIEW 2.9). ARMn_SENSE = the same from each fused bus."
- note removed: "D120 + R131/R143 (10k): cold pull-up of both drains (FMEA H-1) for plug-out FET-short detection. In flight: log only, never veto (F-10)."
- note removed: "Igniter 1 across J121.1-2, igniter 2 across J125.1-2. Each pin order is reversal-symmetric within its channel."
- note removed: "Pass 11: each divider top is 2 x 5.1k in series (R173 + R129, R174 + R141 from the drains; R132 + R175, R144 + R176 from the buses); pass 12: each bottom is 2 x 2k in parallel (R130 + R178, R142 + R179, R133 + R180, R145 + R181). Ratio 1/11.2. One shorted or open 0402 leaves its ADC node <= 1.4 V (<= 3.3 V at the 19.9 V clamp) and the igniter <= 1.4 mA; R168-R171 (4.7k at the MCU pins) stay as th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"
- note removed: "R134/R135: 2 ohm 2 W pulse-rated (Bourns CRM2512, 90 W for 10 ms). Limit a shorted igniter to ~4 A so BAT_IN, the MCU and the other channel survive (m3_design/sim_r2/FINDINGS.md 1). Firmware fire pulse <= 20 ms."
- note removed: "Two independent channels (FMEA H-5). ARM links: J124.2 (RAW) -> F1 5A FAST -> J124.1 (BUS1); J120.1 (RAW) -> F2 5A FAST -> J120.2 (BUS2). R4: DB128L 2P pairs, ARM terminals black, igniter terminals orange."
- note removed: "With the plug out NOTHING connects RAW_ACT to PYRO1_BUS or PYRO2_BUS (AGENTS.md safety rule 1). No test point on BUS/OUT."
- title: 12 | Pyro channels, arming and continuity -> 12 | Single pyro CH1, arming and continuity
