File: m3_design/assembly_review/pyro.kicad_sch (KiCad schematic)
At the start: 22 parts, among them J121 IGNITER 1: E1- / E1+, J124 ARM CH1: BUS1 / RAW, Q124 AON7524

Commit message: M3-ASSY-R9: clean-sheet B-spine layout, 46 x 102 mm, owner-accepted deviations
R8's circuit laid out again from a clean sheet (r9_plan.md): the RF strip aft,
the CH1 pyro column as a dead end on the west edge, all power in the east
column. Built reproducibly from R8's sources by m3_design/r9_build.sh and
judged by the rule-based gate tools/check_r9.py; route_check profile r9 has an
empty allowlist and no leftovers. Every safety and RF qualification is
re-derived on the final board 4f841a0e (docs/R9_VALIDATION.md).

Review passes 1 and 2 found no confirmed Critical or Major; pass 1's Minors
were fixed through the generators, pass 2's 32 Minors are recorded. The owner
accepted the R9 deviation list on 2026-10-25, including the IMU turned 180
degrees (roll = -gyro_Y) and the crystal's local In2 GND plane, and kept the
board at 102 mm. tools/check.sh exits 0. R8 stays the accepted fallback.

Co-Authored-By: Claude Opus 5.5 <noreply@anthropic.com>
Parts:
- J121, J124: footprint rocket:M3_DB128L_2P_BK -> rocket:M3_DB128L_2P_BK_SW
Other:
- note added: "Igniter across J121.1 OUT and J121.2 IGN. J124 and J121 pin numbering (the net on each pin) is retained from the reviewed CH1. R9: both on M3_DB128L_2P_BK_SW (the DB128L with pads 1 and 2 swapped: same part C430601, same land), turned so both wires enter from -x (pyro leads west) with pin 2 (RAW / IGN) forward and pin 1 (BUS / OUT) aft."
- note removed: "Igniter across J121.1 OUT and J121.2 IGN. J124 and J121 pin ordering is retained from the reviewed CH1."
Changed lines of the file:
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@@
 		(title "12 | Single pyro CH1, arming and continuity")
 		(date "2026-09-25")
-		(rev "M3-ASSY-R8")
+		(rev "M3-ASSY-R9")
 		(company "Single-board M3 candidate; actuator merge, not bench-verified"))
 	(symbol
@@
 					(size 1.27 1.27))
 				(justify left)))
-		(property "Footprint" "rocket:M3_DB128L_2P_BK"
+		(property "Footprint" "rocket:M3_DB128L_2P_BK_SW"
 			(at 332.74 243.84 0)
 			(hide yes)
@@
 					(size 1.27 1.27))
 				(justify left)))
-		(property "Footprint" "rocket:M3_DB128L_2P_BK"
+		(property "Footprint" "rocket:M3_DB128L_2P_BK_SW"
 			(at 391.16 238.76 0)
 			(hide yes)
@@
 			(justify left))
 )
-	(text "Igniter across J121.1 OUT and J121.2 IGN. J124 and J121 pin ordering is retained from the reviewed CH1."
+	(text "Igniter across J121.1 OUT and J121.2 IGN. J124 and J121 pin numbering (the net on each pin) is retained from the reviewed CH1. R9: both on M3_DB128L_2P_BK_SW (the DB128L with pads 1 and 2 swapped: same part C430601, same land), turned so both wires enter from -x (pyro leads west) with pin 2 (RAW / IGN) forward and pin 1 (BUS / OUT) aft."
 		(at 20.32 345.24 0)
 		(effects
