File: m3_design/assembly_review/usb_sense.kicad_sch (KiCad schematic)
At the start: 3 parts

Commit message: Validate and harden R5 flight computer CAD
Parts:
- R9: Manufacturer (none) -> UNI-ROYAL(Uniroyal Elec); Manufacturer Part (none) -> 0402WGF1001TCE
Changed lines of the file:
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@@
 					(reference "R9")
 					(unit 1))))
-		(property "Manufacturer" ""
+		(property "Manufacturer" "UNI-ROYAL(Uniroyal Elec)"
 			(at 78.74 83.82 0)
 			(hide yes)
@@
 				(font
 					(size 1.27 1.27))))
-		(property "Manufacturer Part" ""
+		(property "Manufacturer Part" "0402WGF1001TCE"
 			(at 78.74 83.82 0)
 			(hide yes)
