File: m3_design/assembly_review/telemetry.kicad_sch (KiCad schematic)
At the start: 26 parts, among them J410 GPS 4V8/GND/TX/RX, J420 RADIO 4V8/GND/TX/RX, U411 TXU0202DCUR, U412 TPS70933DBVR, U421 TXU0202DCUR, U422 TPS70933DBVR

Commit message: R10 requirements-audit cuts and GAP fixes before review round 9
Implement adopted AUD-1 through AUD-10 and GAP-1 through GAP-5 after the single-switch pass.
Remove the advisory pull-pin, redundant probes and GPS/radio IO LDO cells; qualify the smaller
AONR21357 pair, correct C120 voltage rating, standardize shared-code capacitor lands, simplify
slow returns and fire-only copper, localize U9 output protection and add exactly two U401 VIPPO vias.
Record physical-current timing, coupled fire/source budget, C84 manual fitting and narrowed gate scopes.

Board SHA-256: 877d01996a59e9dd5c6dbc367274bb9a323a13982d67960fe46df9b0ee53205d
Board: 46 x 90 mm, 4 layers, 2365477 bytes; 225 footprints, 883 straight tracks, 323 vias.
Netlist SHA-256: 0843da709e2d7a757e9b35cdff48158a54012c5353619cbf409ab961efd2c3ca
Two fresh complete passing builds are byte-identical. Schematic: 700 pins; 22 seeded faults detected.

Final unskipped tools/check.sh: exit 0
DRC violations 0  unconnected 0  schematic parity 0  ERC 0
metadata / 3D model audit: OK
silkscreen outside the board outline: 0 stroke points
fit check: OK (CAD envelopes only)
R10 CAD contract (full): OK
routing hygiene: 0 failing, 0 allowlisted, 0 leftovers recorded
actuator safety contract: OK
Fab manifest: OK; 5 outputs match current CAD and export inputs
Self-tests: shell 4, fit 24, paste 5, routing 59, R10 131; three NumPy cases rerun and passed.

Fab: 215 CPL rows, 82 BOM codes; orientation / paste / manifest pass. Hot-plug: 2304 required
cases plus convergence and controls pass (simulation / Inference). Plate f1 280.9 Hz (Inference).
Live JLC: $84.43 vs $84.41 target, 46 Extended codes; R430 / U4 short. Procurement exit 1 is a
disclosed OQ-3 / ordering deviation, not a CAD gate pass. No quote accepted or order placed.
Firmware, bench, thermal/transient correlation, process acceptance, installed RF immunity and physical fit unverified.

This preparatory pass earns no clean-review credit. Start fresh full ten-lens round 9 on th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
Parts:
- removed C441, C451: 1uF 50V X7R 10%, rocket:C_1206_3216Metric, symbol M3:C
- removed C442, C452: 22uF 25V X7R 10%, rocket:M3_GRM32_1210, symbol M3:C
- removed R443, R453: 1k 1%, rocket:R_0603_1608Metric, symbol M3:R
- removed U412, U422: TPS70933DBVR, rocket:M3_TPS709_DBV, symbol M3:CameraUARTSupply
Connections:
- net GPS_IO_3V3 is gone; now on net 3V3: C443.1, U411.7 (VCCB CAMERA)
- net RADIO_IO_3V3 is gone; now on net 3V3: C453.1, U421.7 (VCCB CAMERA)
- no-connect marks 4 -> 0
Other:
- note added: "Reset / boot / port off: EN=0 and OE=0. Startup: EN, stable downstream supply, UART idle-high configuration, then OE. Shutdown: OE low before EN low. Incorrect OE while port off may feed a few mA through 1k; accepted."
- note added: "TXU0202 VCCA and VCCB = main 3V3; C440/C450 and retained C443/C453 bypass the two supplies. OE has 10k pull-down. 1k UART series resistors and ground-only ESD clamps remain."
- note removed: "Reset / boot / off: EN=0 and OE=0. Startup: EN, stable downstream supply, UART idle-high configuration, then OE. Shutdown: OE low before EN low."
- note removed: "TXU0202 VCCA = main 3V3, VCCB = own switched TPS70933 output. OE has 10k pull-down. 1k UART series resistors and ground-only ESD clamps."
- moved on the sheet: C440, C443, C450, C453, D410, D411, D420, D421, J420, R440, R441, R442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
